File: pcb/ad9866.sch (KiCad schematic (older format))
At the start: 71 parts, among them CN1 MEC6-140_CONNECTOR_BEMICRO, CN2 PCIE, P1 CONN_4, P10 CONN_1, P13 CONN_1, P14 CONN_1, P15 Si510 73.728, P16 CONN_3X2, P17 CONN_4, P18 CONN_1, P19 CONN_1, P2 CONN_1, P20 CONN_1, P22 CONN_1, P23 CONN_5, P24 CONN_5, P25 CONN_5, P3 CONN_1, P4 CONN_1, P5 CONN_1, P6 CONN_1, P8 CONN_1, P9 CONN_1, T1 TRANSF_ADT8, T2 TRANSF_ADT2, T3 TRANSF_ADT2, U1 AD9866BCPZ, U2 NCP1117ST33T3G, U3 NCP1117ST33T3G

Commit message: Schematic rev 1.1a
Parts:
- removed C23, C24, C28, C29: 0.1UF, symbol CSMALL
- removed C25: 10UF, symbol CSMALL
- removed P1, P17: CONN_4, symbol CONN_4
- removed P10, P13, P14, P18, P19, P2, P20, P22, P3, P4, P5, P6, P8, P9: CONN_1, symbol CONN_1
- removed P16: CONN_3X2, symbol CONN_3X2
- removed P23: CONN_5, symbol CONN_5
- removed T2: TRANSF_ADT2, symbol TRANSF_ADT2
- removed U2, U3: NCP1117ST33T3G, symbol NCP1117ST33T3G
- added C23, C24, C28, C29, C31, C32: 0.1UF, symbol Csmall
- added C25: 10UF, symbol Csmall
- added L5: FB, symbol INDUCTOR_SMALL
- added P1: DIL20, symbol DIL20
- added P16: DIPSW, symbol dipswitch
- added P2: CONN_15, symbol CONN_15
- added R10, R11, R8, R9: 0, symbol R
- added R12: 200, symbol R
- C1, C10, C11, C12, C13, C14, C15, C16, C2, C21, C26, C27, C3, C30, C4, C5, C6, C7, C8, C9: symbol CSMALL -> Csmall
- C17, C18, C19, C20, C22: symbol CPSMALL -> CPsmall
- P15: value Si510 73.728 -> 61.440
- R1: value 10K -> 0
- R6, R7: value DNI -> 0
- T1: value TRANSF_ADT8 -> 8:1
- T3: value TRANSF_ADT2 -> 4:1
Connections:
- net labels added: 12VIN, 3VIN, 5VIN, TXLN, TXLP, TXN, TXP
- net labels removed: SCLK, SDIO, SDO, SEN, VIN
- wire segments 332 -> 286
- no-connect marks 0 -> 7
Other:
- moved on the sheet: CN1, CN2, D1, L1, L2, L3, L4, P15, P24, P25, R2, R3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

Commit message: Before library and name changes
Parts:
- removed L1, L2, L3, L4, L5: FB, symbol INDUCTOR_SMALL
- removed P24, P25: CONN_5, symbol CONN_5
- added L1, L2, L3, L4, L5: FB, symbol FB
- added P24, P25: BNC, symbol BNC
- added P? (x5): CONN_1, symbol CONN_1
- added R? (x2): R, symbol R
Connections:
- net 12VIN: now also P?.1
- net 3VIN: now also L1.1, L2.1, L3.1, L4.1, P?.1
- net 5VIN: now also L5.1, P?.1; no longer C26.1, R6.1, T3.5 (PM)
- net AVDD_ADC: now also L1.2
- net AVDD_DAC: now also L2.2
- net CLKVDD: now also L3.2
- net DVDD: now also L4.2
- net GND: now also CN2.B2, CN2.B3, CN2.B5, CN2.B6, CN2.B8, CN2.B9, P24.2 (Ext), P25.2 (Ext), P?.1, R?.2; no longer CN1.4 (PWREN#), CN2.A2, CN2.A3, CN2.A5, CN2.A6, CN2.A8, CN2.A9
- net RXN: now also CN2.A2; no longer CN2.B2
- net RXP: now also CN2.A3; no longer CN2.B3
- net TXLN: now also CN2.A8; no longer CN2.B8
- net TXLP: now also CN2.A9; no longer CN2.B9
- net TXN: now also CN2.A5; no longer CN2.B5
- net TXP: now also CN2.A6; no longer CN2.B6
- net at CN1.6 (P35): now also U1.16 (RXCLK); no longer U1.19 (CLKOUT1)
- net at C30.2: now also P25.1 (In)
- net at C22.1, R6.2: now also L5.2
- net at T3.1 (S2): now also P24.1 (In)
- net at CN1.1 (3V3): now also CN1.2 (3V3), P?.1
- net at CN1.50 (P53): now also CN2.B14; no longer CN2.A14
- net at CN1.52 (P54): now also CN2.B15; no longer CN2.A15
- net at CN1.56 (P55): now also CN2.B16; no longer CN2.A16
- net at CN1.58 (P56): now also CN2.B17; no longer CN2.A17
- net at CN1.60 (P57): now also CN2.A17; no longer CN2.B17
- net at CN1.62 (P58): now also CN2.A16; no longer CN2.B16
- net at CN1.64 (P59): now also CN2.A15; no longer CN2.B15
- net at CN1.66 (P60): now also CN2.A14; no longer CN2.B14
- net at CN1.7 (P2): now also P1.14 (P14); no longer P1.13 (P13)
- net at CN1.9 (P3): now also P1.13 (P13); no longer P1.14 (P14)
- new net: R1.2, R?.1, U1.19 (CLKOUT1)
- new net: C26.1, R6.1, T3.5 (PM)
- new net: CN1.4 (PWREN#), R?.1
- new net: CN1.5 (P1), R?.2
- no-connect marks 7 -> 5
