File: pcb/hermeslite.sch (KiCad schematic (older format))
At the start: 79 parts, among them CN1 MEC6-140_CONNECTOR_BEMICRO, CN2 PCIE, CN3 GPIO, CN4 POWER, J1 0, J2 0, J3 0, J4 0, J5 0, J6 0, J7 0, J8 0, P0 CONN_1, P1 CONN_1, P12 CONN_1, P3 CONN_1, P5 CONN_1, U1 AD9866BCPZ, U2 EEPROM, X1 61.440

Commit message: Update to v1.22
Parts:
- X1: value 61.440 -> 73.728
Connections:
- wire segments 302 -> 304
Other:
- moved on the sheet: X1
Changed lines of the file:
@@
 Sheet 1 1
 Title "Hermes-Lite"
-Date "07 Dec 2014"
-Rev "1.21"
+Date "22 May 2015"
+Rev "1.22"
 Comp "SofterHardware"
 Comment1 "KF7O Steve Haynal"
@@
 L CONN_4 X1
 U 1 1 52D1F475
-P 3600 2250
-F 0 "X1" V 3550 2250 50  0000 C CNN
-F 1 "61.440" V 3650 2250 50  0000 C CNN
-F 2 "HERMESLITE:Si510" H 3600 2250 60  0001 C CNN
-F 3 "" H 3600 2250 60  0000 C CNN
-	1    3600 2250
-	-1   0    0    1
-$EndComp
-Text GLabel 3950 2100 2    60   Input ~ 0
+P 4300 1750
+F 0 "X1" V 4250 1750 50  0000 C CNN
+F 1 "73.728" V 4350 1750 50  0000 C CNN
+F 2 "HERMESLITE:Si510" H 4300 1750 60  0001 C CNN
+F 3 "" H 4300 1750 60  0000 C CNN
+	1    4300 1750
+	0    1    -1   0
+$EndComp
+Text GLabel 4050 2100 0    60   Input ~ 0
 CLKVDD
-$Comp
-L GND #PWR04
-U 1 1 52D1F5D4
-P 4100 2450
-F 0 "#PWR04" H 4100 2450 30  0001 C CNN
-F 1 "GND" H 4100 2380 30  0001 C CNN
-F 2 "" H 4100 2450 60  0000 C CNN
-F 3 "" H 4100 2450 60  0000 C CNN
-	1    4100 2450
-	1    0    0    -1
-$EndComp
 $Comp
 L PCIE CN2
@@
 $EndComp
 $Comp
-L GND #PWR012
-U 1 1 5420DCD7
-P 4350 2250
-F 0 "#PWR012" H 4350 2250 30  0001 C CNN
-F 1 "GND" H 4350 2180 30  0001 C CNN
-F 2 "" H 4350 2250 60  0000 C CNN
-F 3 "" H 4350 2250 60  0000 C CNN
-	1    4350 2250
-	0    1    1    0
-$EndComp
-$Comp
 L Csmall C33
 U 1 1 54222EC4
@@
 U 1 1 54287617
 P 3300 2500
-F 0 "TP2" H 3150 2550 40  0000 L CNN
+F 0 "TP2" H 3350 2550 40  0000 L CNN
 F 1 "CONN_1" H 3300 2555 30  0001 C CNN
 F 2 "HERMESLITE:TP" H 3300 2500 60  0001 C CNN
@@
 Connection ~ 5100 7000
 Wire Wire Line
-	3950 2200 4200 2200
-Wire Wire Line
-	4200 2200 4200 2450
-Wire Wire Line
-	3950 2300 4100 2300
-Wire Wire Line
-	4100 2300 4100 2450
-Wire Wire Line
-	3950 2400 4100 2400
-Connection ~ 4100 2400
-Wire Wire Line
 	1550 1900 1550 1700
 Wire Wire Line
@@
 Connection ~ 3300 7150
 Wire Wire Line
-	4450 2150 4450 2350
-Wire Wire Line
-	4450 2250 4350 2250
-Connection ~ 4450 2250
-Wire Wire Line
 	1550 5300 1250 5300
 Wire Wire Line
@@
 Wire Wire Line
 	6950 4750 7000 4750
-Wire Wire Line
-	4200 2450 4450 2450
 Connection ~ 1500 5400
 Wire Wire Line
@@
 Wire Wire Line
 	6450 2000 6450 3250
+Wire Wire Line
+	4250 2100 4250 2450
+Wire Wire Line
+	4250 2450 4450 2450
+Wire Wire Line
+	4350 2100 4450 2100
+Wire Wire Line
+	4450 2100 4450 2150
+Connection ~ 4450 2100
+Wire Wire Line
+	4050 2100 4150 2100
+Wire Wire Line
+	4450 2250 3150 2250
+Wire Wire Line
+	3150 2250 3150 2500
+Connection ~ 3150 2500
+Wire Wire Line
+	4350 2100 4350 2350
+Wire Wire Line
+	4150 2350 4450 2350
+Connection ~ 4350 2100
+$Comp
+L GND #PWR?
+U 1 1 556021D1
+P 4150 2400
+F 0 "#PWR?" H 4150 2400 30  0001 C CNN
+F 1 "GND" H 4150 2330 30  0001 C CNN
+F 2 "" H 4150 2400 60  0000 C CNN
+F 3 "" H 4150 2400 60  0000 C CNN
+	1    4150 2400
+	1    0    0    -1
+$EndComp
+Wire Wire Line
+	4150 2350 4150 2400
+Connection ~ 4350 2350
 $EndSCHEMATC
