File: frontend/basic/frontend.kicad_pcb (KiCad board)
At the start: 2 copper layers, 41.5 x 49.9 mm, 69 parts, among them CN1 EDGE, CN2 BREAKOUT, CN3 CONN_01X02, CN4 CONN_01X02, CN5 CONN_01X02, CN6 CONN_01X02, CN7 CONN_01X02, J1 0, J2 0, P1 BNC, P2 BNC, P5 CONN_01X10, Q1 2N3904, Q2 2N7002, T1 1.8:1, T2 9:1, U1 ULN2003A

Commit message: Revert "Added UNL2003 and connectors"
Parts:
- removed CN6, CN7: CONN_01X02, Pin_Headers:Pin_Header_Straight_1x02
- removed the HOLE at (129.6, 81.2)
- removed the HOLE at (127.0, 81.2)
- removed the HOLE at (124.5, 81.2)
- removed the HOLE at (121.9, 81.2)
- removed the HOLE at (127.0, 83.8)
- removed the HOLE at (134.6, 86.3)
- removed P5: CONN_01X10, Pin_Headers:Pin_Header_Straight_1x10
- removed Q1: 2N3904, SMD_Packages:SOT-23
- removed Q2: 2N7002, SMD_Packages:SOT-23-GDS
- removed R2, R3: 4.99k, SMD_Packages:SMD-0805
- removed U1: ULN2003A, Housings_SOIC:SOIC-16_7.5x10.3mm_Pitch1.27mm
- added HOLE: VAL**, HERMESLITE:HOLE, F.Cu at (101.6, 81.3)
- added HOLE: VAL**, HERMESLITE:HOLE, F.Cu at (109.2, 81.3)
- added HOLE: VAL**, HERMESLITE:HOLE, F.Cu at (111.8, 81.3)
- added HOLE: VAL**, HERMESLITE:HOLE, F.Cu at (114.3, 81.3)
- added HOLE: VAL**, HERMESLITE:HOLE, F.Cu at (116.8, 81.3)
- added HOLE: VAL**, HERMESLITE:HOLE, F.Cu at (119.4, 81.3)
- added HOLE: VAL**, HERMESLITE:HOLE, F.Cu at (121.9, 81.3)
- added HOLE: VAL**, HERMESLITE:HOLE, F.Cu at (124.5, 81.3)
- added HOLE: VAL**, HERMESLITE:HOLE, F.Cu at (127.0, 81.3)
- added HOLE: VAL**, HERMESLITE:HOLE, F.Cu at (129.5, 81.3)
- added HOLE: VAL**, HERMESLITE:HOLE, F.Cu at (116.8, 83.8)
- added HOLE: VAL**, HERMESLITE:HOLE, F.Cu at (114.3, 83.8)
- added HOLE: VAL**, HERMESLITE:HOLE, F.Cu at (104.1, 81.3)
- added HOLE: VAL**, HERMESLITE:HOLE, F.Cu at (119.4, 83.8)
- added HOLE: VAL**, HERMESLITE:HOLE, F.Cu at (121.9, 83.8)
- added HOLE: VAL**, HERMESLITE:HOLE, F.Cu at (124.5, 83.8)
- added HOLE: VAL**, HERMESLITE:HOLE, F.Cu at (127.0, 83.8)
- added HOLE: VAL**, HERMESLITE:HOLE, F.Cu at (132.1, 86.4)
- added HOLE: VAL**, HERMESLITE:HOLE, F.Cu at (129.5, 86.4)
- added HOLE: VAL**, HERMESLITE:HOLE, F.Cu at (127.0, 86.4)
- added HOLE: VAL**, HERMESLITE:HOLE, F.Cu at (124.5, 86.4)
- added HOLE: VAL**, HERMESLITE:HOLE, F.Cu at (121.9, 86.4)
- added HOLE: VAL**, HERMESLITE:HOLE, F.Cu at (119.4, 86.4)
- added HOLE: VAL**, HERMESLITE:HOLE, F.Cu at (116.8, 86.4)
- added HOLE: VAL**, HERMESLITE:HOLE, F.Cu at (116.8, 88.9)
- added HOLE: VAL**, HERMESLITE:HOLE, F.Cu at (119.4, 88.9)
- added HOLE: VAL**, HERMESLITE:HOLE, F.Cu at (121.9, 88.9)
- added HOLE: VAL**, HERMESLITE:HOLE, F.Cu at (124.5, 88.9)
- added HOLE: VAL**, HERMESLITE:HOLE, F.Cu at (127.0, 88.9)
- added HOLE: VAL**, HERMESLITE:HOLE, F.Cu at (129.5, 88.9)
- added HOLE: VAL**, HERMESLITE:HOLE, F.Cu at (132.1, 88.9)
- added HOLE: VAL**, HERMESLITE:HOLE, F.Cu at (132.1, 91.4)
- added HOLE: VAL**, HERMESLITE:HOLE, F.Cu at (129.5, 91.4)
- added HOLE: VAL**, HERMESLITE:HOLE, F.Cu at (127.0, 91.4)
- added HOLE: VAL**, HERMESLITE:HOLE, F.Cu at (124.5, 91.4)
- added HOLE: VAL**, HERMESLITE:HOLE, F.Cu at (121.9, 91.4)
- added HOLE: VAL**, HERMESLITE:HOLE, F.Cu at (119.4, 91.4)
- added HOLE: VAL**, HERMESLITE:HOLE, F.Cu at (116.8, 91.4)
- added HOLE: VAL**, HERMESLITE:HOLE, F.Cu at (114.3, 91.4)
- added HOLE: VAL**, HERMESLITE:HOLE, F.Cu at (106.7, 81.3)
- added HOLE: VAL**, HERMESLITE:HOLE, F.Cu at (134.6, 86.4)
- added HOLE: VAL**, HERMESLITE:HOLE, F.Cu at (134.6, 88.9)
- added HOLE: VAL**, HERMESLITE:HOLE, F.Cu at (134.6, 91.4)
- added HOLE: VAL**, HERMESLITE:HOLE, F.Cu at (116.8, 94.0)
- added HOLE: VAL**, HERMESLITE:HOLE, F.Cu at (119.4, 94.0)
- added HOLE: VAL**, HERMESLITE:HOLE, F.Cu at (121.9, 94.0)
- added HOLE: VAL**, HERMESLITE:HOLE, F.Cu at (124.5, 94.0)
- added HOLE: VAL**, HERMESLITE:HOLE, F.Cu at (127.0, 94.0)
- added HOLE: VAL**, HERMESLITE:HOLE, F.Cu at (129.5, 94.0)
- added HOLE: VAL**, HERMESLITE:HOLE, F.Cu at (132.1, 94.0)
- added HOLE: VAL**, HERMESLITE:HOLE, F.Cu at (134.6, 94.0)
- added HOLE: VAL**, HERMESLITE:HOLE, F.Cu at (124.5, 96.5)
- added HOLE: VAL**, HERMESLITE:HOLE, F.Cu at (127.0, 96.5)
- added HOLE: VAL**, HERMESLITE:HOLE, F.Cu at (129.5, 96.5)
- added HOLE: VAL**, HERMESLITE:HOLE, F.Cu at (132.1, 96.5)
- added HOLE: VAL**, HERMESLITE:HOLE, F.Cu at (134.6, 96.5)
- added HOLE: VAL**, HERMESLITE:HOLE, F.Cu at (127.0, 99.1)
- added HOLE: VAL**, HERMESLITE:HOLE, F.Cu at (129.5, 99.1)
- added HOLE: VAL**, HERMESLITE:HOLE, F.Cu at (132.1, 99.1)
- added HOLE: VAL**, HERMESLITE:HOLE, F.Cu at (134.6, 99.1)
- added HOLE: VAL**, HERMESLITE:HOLE, F.Cu at (129.5, 101.6)
- added HOLE: VAL**, HERMESLITE:HOLE, F.Cu at (132.1, 101.6)
- added HOLE: VAL**, HERMESLITE:HOLE, F.Cu at (134.6, 101.6)
- added HOLE: VAL**, HERMESLITE:HOLE, F.Cu at (134.6, 104.1)
- added HOLE: VAL**, HERMESLITE:HOLE, F.Cu at (134.6, 106.7)
- added HOLE: VAL**, HERMESLITE:HOLE, F.Cu at (134.6, 109.2)
- added HOLE: VAL**, HERMESLITE:HOLE, F.Cu at (134.6, 111.8)
- CN3: value CONN_01X02 -> TXL
- CN4, CN5: value CONN_01X02 -> AGND
- T1: value 1.8:1 -> 4:1
- T2: value 9:1 -> 8:1
- moved CN3 6.60 mm to (103.0, 94.7), turned to 270 degrees
- moved CN4 4.07 mm to (130.8, 104.9), turned to 90 degrees
Connections:
- CN3 pad 1: Net-(CN1-PadB8) -> Net-(CN1-PadB9)
- CN3 pad 2: Net-(CN1-PadB9) -> Net-(CN1-PadB8)
Routing:
- net Net-(CN1-PadB14): track 40.3 -> 7.22 mm, vias 1 -> 0
- net GND: track 97.4 -> 65.5 mm, vias 9 -> 3
- net Net-(CN1-PadB15): track 37.3 -> 7.61 mm, vias 1 -> 0
- net Net-(CN1-PadB16): track 37.6 -> 11.0 mm, vias 1 -> 0
- net Net-(CN1-PadB13): track 36.9 -> 11.2 mm, vias 1 -> 0
- net Net-(CN1-PadB17): track 37.3 -> 13.7 mm, vias 1 -> 0
- net Net-(CN1-PadB18): track 37.7 -> 16.3 mm, vias 1 -> 0
- net Net-(CN1-PadB11): track 36.3 -> 16.7 mm
- net Net-(CN1-PadB12): track 31.6 -> 13.5 mm, vias 1 -> 0
- net Net-(P5-Pad9): track 17.4 -> 0.00 mm
- net Net-(P5-Pad8): track 14.0 -> 0.00 mm
- net Net-(P5-Pad7): track 14.0 -> 0.00 mm
- net Net-(P5-Pad6): track 12.5 -> 0.00 mm
- net Net-(P5-Pad5): track 11.0 -> 0.00 mm
- net Net-(P5-Pad4): track 9.95 -> 0.00 mm
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- added copper zone on B.Cu, net Net-(D1-Pad2)
- added copper zone on F.Cu, net Net-(D1-Pad2)
- added copper zone on B.Cu, net Net-(J1-Pad1)
- added copper zone on F.Cu, net Net-(J1-Pad1)
- removed copper zone on B.Cu, net Net-(D1-Pad2) (its old number)
- removed copper zone on F.Cu, net Net-(D1-Pad2) (its old number)
- removed copper zone on B.Cu, net Net-(J1-Pad1) (its old number)
- removed copper zone on F.Cu, net Net-(J1-Pad1) (its old number)
