File: frontend/basic/frontend.sch (KiCad schematic (older format))
At the start: 26 parts, among them CN1 EDGE, CN2 BREAKOUT, CN3 TXL, CN4 AGND, CN5 AGND, J1 0, J2 0, P1 BNC, P2 BNC, P3 CONN_01X02, P4 CONN_01X02, P5 CONN_01X10, Q1 2N3904, Q2 2N7002, T1 1.8:1, T2 9:1, U1 ULN2003A

Commit message: Revert "Added UNL2003 and connectors"
Parts:
- removed P3, P4: CONN_01X02, symbol CONN_01X02
- removed P5: CONN_01X10, symbol CONN_01X10
- removed Q1: 2N3904, symbol NPN
- removed Q2: 2N7002, symbol MOSFET_N
- removed R2, R3: 4.99k, symbol R
- removed U1: ULN2003A, symbol ULN2003A
Connections:
- wire segments 135 -> 86
Other:
- note removed: "7 Open Collector User Outputs\n(based on Hermes J16)\nPin 8 Open Collector Reference/fly-back Diodes\nPin 9 Open Drain PTT\nAll require pull up resistors"
- moved on the sheet: CN2
