File: frontend/basic/$frontend.sch (KiCad schematic (older format))
At the start: 26 parts, among them CN1 EDGE, CN2 BREAKOUT, CN3 TXL, CN4 AGND, CN5 AGND, J1 0, J2 0, P1 BNC, P2 BNC, P3 CONN_01X02, P4 CONN_01X02, P5 CONN_01X10, Q1 2N3904, Q2 2N7002, T1 1.8:1, T2 9:1, U1 ULN2003A

Commit message: Added UNL2003 and connectors
Parts:
- removed CN3: TXL, symbol CONN_2
- removed CN4, CN5: AGND, symbol CONN_2
- added CN3, CN4, CN5: CONN_01X02, HERMESLITE:JUMPER, symbol CONN_01X02
- C1, C2, C3, C4, FB1, R1, R2, R3: footprint (none) -> SMD_Packages:SMD-0805
- CN1: footprint (none) -> HERMESLITE:EDGE
- CN2: footprint (none) -> HERMESLITE:BREAKOUT
- CN6: renamed from P3; footprint (none) -> Pin_Headers:Pin_Header_Straight_1x02
- CN7: renamed from P4; footprint (none) -> Pin_Headers:Pin_Header_Straight_1x02
- D1: footprint (none) -> HERMESLITE:SOD323
- J1, J2: footprint (none) -> HERMESLITE:JUMPER
- P1, P2: footprint (none) -> HERMESLITE:BNCRA
- P5: footprint (none) -> Pin_Headers:Pin_Header_Straight_1x10
- Q1: footprint (none) -> SMD_Packages:SOT-23
- Q2: footprint (none) -> SMD_Packages:SOT-23-GDS
- T1, T2: footprint (none) -> HERMESLITE:TRANSFREV
- U1: footprint (none) -> Housings_SOIC:SOIC-16_7.5x10.3mm_Pitch1.27mm
Connections:
- wire segments 135 -> 137
Other:
- note added: "CN6 and CN7 provided for molex style connection to \nMegaboard amp in lieu of BNC connectors"
- moved on the sheet: R3
Changed lines of the file:
@@
 F 0 "CN1" H 3250 2450 60  0000 C CNN
 F 1 "EDGE" H 3250 4500 60  0000 C CNN
-F 2 "" H 3250 3100 60  0000 C CNN
+F 2 "HERMESLITE:EDGE" H 3250 3100 60  0001 C CNN
 F 3 "" H 3250 3100 60  0000 C CNN
 	1    3250 3600
@@
 F 0 "T2" H 5700 4150 70  0000 C CNN
 F 1 "9:1" H 5700 4750 70  0000 C CNN
-F 2 "" H 5700 4450 60  0000 C CNN
+F 2 "HERMESLITE:TRANSFREV" H 5700 4450 60  0001 C CNN
 F 3 "" H 5700 4450 60  0000 C CNN
 	1    5700 4450
@@
 F 0 "T1" H 5700 2700 70  0000 C CNN
 F 1 "1.8:1" H 5700 3300 70  0000 C CNN
-F 2 "" H 5700 3000 60  0000 C CNN
+F 2 "HERMESLITE:TRANSFREV" H 5700 3000 60  0001 C CNN
 F 3 "" H 5700 3000 60  0000 C CNN
 	1    5700 3000
@@
 F 0 "P1" H 7260 2920 60  0000 C CNN
 F 1 "BNC" H 7350 2700 40  0000 C CNN
-F 2 "" H 7250 2800 60  0000 C CNN
+F 2 "HERMESLITE:BNCRA" H 7250 2800 60  0001 C CNN
 F 3 "" H 7250 2800 60  0000 C CNN
 	1    7250 2800
@@
 F 0 "P2" H 7260 4370 60  0000 C CNN
 F 1 "BNC" H 7350 4150 40  0000 C CNN
-F 2 "" H 7250 4250 60  0000 C CNN
+F 2 "HERMESLITE:BNCRA" H 7250 4250 60  0001 C CNN
 F 3 "" H 7250 4250 60  0000 C CNN
 	1    7250 4250
@@
 F 0 "C3" V 6350 4150 30  0000 L CNN
 F 1 "0.1 uF" V 6350 4300 30  0000 L CNN
-F 2 "" H 6400 4250 60  0000 C CNN
+F 2 "SMD_Packages:SMD-0805" H 6400 4250 60  0001 C CNN
 F 3 "" H 6400 4250 60  0000 C CNN
 	1    6400 4250
@@
 F 0 "C4" V 6750 4150 30  0000 L CNN
 F 1 "0.1 uF" V 6750 4300 30  0000 L CNN
-F 2 "" H 6800 4250 60  0000 C CNN
+F 2 "SMD_Packages:SMD-0805" H 6800 4250 60  0001 C CNN
 F 3 "" H 6800 4250 60  0000 C CNN
 	1    6800 4250
@@
 F 0 "C2" H 5125 4950 30  0000 L CNN
 F 1 "0.1 uF" H 5125 4850 30  0000 L CNN
-F 2 "" H 5100 4900 60  0000 C CNN
+F 2 "SMD_Packages:SMD-0805" H 5100 4900 60  0001 C CNN
 F 3 "" H 5100 4900 60  0000 C CNN
 	1    5100 4900
@@
 F 0 "D1" V 6600 4650 40  0000 C CNN
 F 1 "DIODESCH2" H 6600 4275 40  0001 C CNN
-F 2 "" H 6600 4525 60  0000 C CNN
+F 2 "HERMESLITE:SOD323" H 6600 4525 60  0001 C CNN
 F 3 "" H 6600 4525 60  0000 C CNN
 	1    6600 4450
@@
 F 0 "J2" V 6600 4850 40  0000 C CNN
 F 1 "0" V 6600 5050 40  0000 C CNN
-F 2 "" V 6530 4950 30  0000 C CNN
+F 2 "HERMESLITE:JUMPER" V 6530 4950 30  0001 C CNN
 F 3 "" H 6600 4950 30  0000 C CNN
 	1    6600 4950
@@
 F 0 "J1" V 6600 3400 40  0000 C CNN
 F 1 "0" V 6600 3600 40  0000 C CNN
-F 2 "" V 6530 3500 30  0000 C CNN
+F 2 "HERMESLITE:JUMPER" V 6530 3500 30  0001 C CNN
 F 3 "" H 6600 3500 30  0000 C CNN
 	1    6600 3500
@@
 F 0 "R1" V 5100 2600 40  0000 C CNN
 F 1 "0" V 5100 2400 40  0000 C CNN
-F 2 "" V 5030 2500 30  0000 C CNN
+F 2 "SMD_Packages:SMD-0805" V 5030 2500 30  0001 C CNN
 F 3 "" H 5100 2500 30  0000 C CNN
 	1    5100 2500
@@
 F 0 "C1" H 5125 3450 30  0000 L CNN
 F 1 "0.1 uF" H 5125 3350 30  0000 L CNN
-F 2 "" H 5100 3400 60  0000 C CNN
+F 2 "SMD_Packages:SMD-0805" H 5100 3400 60  0001 C CNN
 F 3 "" H 5100 3400 60  0000 C CNN
 	1    5100 3400
@@
 F 0 "FB1" H 4925 2200 39  0000 C CNN
 F 1 "FB" H 4850 2350 60  0001 C CNN
-F 2 "" H 4850 2250 60  0000 C CNN
+F 2 "SMD_Packages:SMD-0805" H 4850 2250 60  0001 C CNN
 F 3 "" H 4850 2250 60  0000 C CNN
 	1    4850 2250
@@
 	2500 3700 2500 4800
 Wire Wire Line
-	2350 3800 2650 3800
+	2100 3800 2650 3800
 Connection ~ 2500 3800
 Wire Wire Line
@@
 Connection ~ 2500 3900
 Wire Wire Line
-	2350 4000 2650 4000
+	2250 4000 2650 4000
 Connection ~ 2500 4000
 Wire Wire Line
@@
 Connection ~ 2500 4100
 Wire Wire Line
-	2350 4200 2650 4200
+	2100 4200 2650 4200
 Connection ~ 2500 4200
 Wire Wire Line
@@
 Connection ~ 2500 4300
 Wire Wire Line
-	2350 4400 2650 4400
+	2250 4400 2650 4400
 Connection ~ 2500 4400
 Wire Wire Line
@@
 F 0 "CN2" V 3600 -200 60  0000 C CNN
 F 1 "BREAKOUT" V 3600 750 60  0000 C CNN
-F 2 "" H 3550 300 60  0000 C CNN
+F 2 "HERMESLITE:BREAKOUT" H 3550 300 60  0001 C CNN
 F 3 "" H 3550 300 60  0000 C CNN
 	1    3550 800
@@
 	2450 2250 4700 2250
 Wire Wire Line
-	3550 1400 3550 2250
-Wire Wire Line
 	2650 3600 2350 3600
 Wire Wire Line
@@
 Wire Wire Line
 	4950 4650 5300 4650
-$Comp
-L CONN_2 CN3
-U 1 1 547563D3
-P 4450 3850
-F 0 "CN3" H 4450 3900 40  0000 C CNN
-F 1 "TXL" H 4450 3800 40  0000 C CNN
-F 2 "" H 4450 3850 60  0000 C CNN
-F 3 "" H 4450 3850 60  0000 C CNN
-	1    4450 3850
-	1    0    0    -1
-$EndComp
-Wire Wire Line
-	3850 3900 4100 3900
-Wire Wire Line
-	4100 3900 4100 3950
-Wire Wire Line
-	3850 3800 4100 3800
-Wire Wire Line
-	4100 3800 4100 3750
-$Comp
-L CONN_2 CN4
-U 1 1 54756604
-P 2000 3900
-F 0 "CN4" H 2000 3850 40  0000 C CNN
-F 1 "AGND" H 2000 3950 40  0000 C CNN
-F 2 "" H 2000 3900 60  0000 C CNN
-F 3 "" H 2000 3900 60  0000 C CNN
-	1    2000 3900
-	-1   0    0    1
-$EndComp
-$Comp
-L CONN_2 CN5
-U 1 1 54756621
-P 2000 4300
-F 0 "CN5" H 2000 4250 40  0000 C CNN
-F 1 "AGND" H 2000 4350 40  0000 C CNN
-F 2 "" H 2000 4300 60  0000 C CNN
-F 3 "" H 2000 4300 60  0000 C CNN
-	1    2000 4300
-	-1   0    0    1
-$EndComp
-$Comp
-L CONN_01X02 P3
+Wire Wire Line
+	3850 3900 4200 3900
+Wire Wire Line
+	3850 3800 4200 3800
+$Comp
+L CONN_01X02 CN6
 U 1 1 54C10BCA
 P 6800 3000
-F 0 "P3" H 6800 3150 50  0000 C CNN
+F 0 "CN6" H 6800 3150 50  0000 C CNN
 F 1 "CONN_01X02" V 6900 3000 50  0001 C CNN
-F 2 "" H 6800 3000 60  0000 C CNN
+F 2 "Pin_Headers:Pin_Header_Straight_1x02" H 6800 3000 60  0001 C CNN
 F 3 "" H 6800 3000 60  0000 C CNN
 	1    6800 3000
@@
 Connection ~ 6600 2800
 $Comp
-L CONN_01X02 P4
+L CONN_01X02 CN7
 U 1 1 54C10FDE
 P 7100 4450
-F 0 "P4" H 7100 4600 50  0000 C CNN
+F 0 "CN7" H 7100 4300 50  0000 C CNN
 F 1 "CONN_01X02" V 7200 4450 50  0001 C CNN
-F 2 "" H 7100 4450 60  0000 C CNN
+F 2 "Pin_Headers:Pin_Header_Straight_1x02" H 7100 4450 60  0001 C CNN
 F 3 "" H 7100 4450 60  0000 C CNN
 	1    7100 4450
@@
 F 0 "U1" H 6750 1400 70  0000 C CNN
 F 1 "ULN2003A" H 6750 1900 70  0000 C CNN
-F 2 "" H 6750 1300 60  0000 C CNN
+F 2 "Housings_SOIC:SOIC-16_7.5x10.3mm_Pitch1.27mm" H 6750 1300 60  0001 C CNN
 F 3 "" H 6750 1300 60  0000 C CNN
 	1    6750 1300
@@
 F 0 "P5" H 8450 1900 50  0000 C CNN
 F 1 "CONN_01X10" V 8550 1350 50  0001 C CNN
-F 2 "" H 8450 1350 60  0000 C CNN
+F 2 "Pin_Headers:Pin_Header_Straight_1x10" H 8450 1350 60  0001 C CNN
 F 3 "" H 8450 1350 60  0000 C CNN
 	1    8450 1350
@@
 F 0 "Q2" H 7450 2300 60  0000 R CNN
 F 1 "2N7002" H 7450 1900 60  0000 R CNN
-F 2 "" H 7500 2100 60  0000 C CNN
+F 2 "SMD_Packages:SOT-23-GDS" H 7500 2100 60  0001 C CNN
 F 3 "" H 7500 2100 60  0000 C CNN
 	1    7500 2100
@@
 Wire Wire Line
 	7600 2300 7600 2400
-Connection ~ 4550 2150
 $Comp
 L NPN Q1
@@
 F 0 "Q1" H 6600 2150 50  0000 R CNN
 F 1 "2N3904" H 6600 2450 50  0000 R CNN
-F 2 "" H 6600 2300 60  0000 C CNN
+F 2 "SMD_Packages:SOT-23" H 6600 2300 60  0001 C CNN
 F 3 "" H 6600 2300 60  0000 C CNN
 	1    6600 2300
@@
 F 0 "R2" V 6050 2400 40  0000 C CNN
 F 1 "4.99k" V 6050 2250 40  0000 C CNN
-F 2 "" V 5980 2300 30  0000 C CNN
+F 2 "SMD_Packages:SMD-0805" V 5980 2300 30  0001 C CNN
 F 3 "" H 6050 2300 30  0000 C CNN
 	1    6050 2300
@@
 $EndComp
 Wire Wire Line
-	4550 2150 5700 2150
-Wire Wire Line
-	5700 2150 5700 2300
+	5700 2100 5700 2300
 Wire Wire Line
 	5700 2300 5800 2300
@@
 L R R3
 U 1 1 54C13EF2
-P 6450 1950
-F 0 "R3" V 6450 2050 40  0000 C CNN
-F 1 "4.99k" V 6450 1900 40  0000 C CNN
-F 2 "" V 6380 1950 30  0000 C CNN
-F 3 "" H 6450 1950 30  0000 C CNN
-	1    6450 1950
+P 6450 1900
+F 0 "R3" V 6450 2000 40  0000 C CNN
+F 1 "4.99k" V 6450 1850 40  0000 C CNN
+F 2 "SMD_Packages:SMD-0805" V 6380 1900 30  0001 C CNN
+F 3 "" H 6450 1900 30  0000 C CNN
+	1    6450 1900
 	0    -1   -1   0
 $EndComp
@@
 	6700 2500 6700 2600
 Wire Wire Line
-	7300 2100 6700 2100
-Wire Wire Line
-	6700 2100 6700 1950
+	6700 2100 7300 2100
+Wire Wire Line
+	6700 1900 6700 2100
 Wire Wire Line
 	7600 1800 7850 1800
@@
 	5700 1750 5700 1500
 Connection ~ 3850 1750
-Wire Wire Line
-	6200 1950 3550 1950
-Connection ~ 3550 1950
 $Comp
 L GND #PWR09
@@
 Wire Wire Line
 	8000 1800 8000 2000
+Text Notes 7400 3800 0    60   ~ 0
+CN6 and CN7 provided for molex style connection to \nMegaboard amp in lieu of BNC connectors
+Wire Wire Line
+	3550 1400 3550 2250
+Wire Wire Line
+	6200 1900 3550 1900
+Connection ~ 3550 1900
+Wire Wire Line
+	4550 2100 5700 2100
+Connection ~ 4550 2100
+$Comp
+L CONN_01X02 CN4
+U 1 1 54C16573
+P 1900 3850
+F 0 "CN4" H 1900 4000 50  0000 C CNN
+F 1 "CONN_01X02" V 2000 3850 50  0001 C CNN
+F 2 "HERMESLITE:JUMPER" H 1900 3850 60  0001 C CNN
+F 3 "" H 1900 3850 60  0000 C CNN
+	1    1900 3850
+	-1   0    0    1
+$EndComp
+$Comp
+L CONN_01X02 CN5
+U 1 1 54C16718
+P 1900 4250
+F 0 "CN5" H 1900 4400 50  0000 C CNN
+F 1 "CONN_01X02" V 2000 4250 50  0001 C CNN
+F 2 "HERMESLITE:JUMPER" H 1900 4250 60  0001 C CNN
+F 3 "" H 1900 4250 60  0000 C CNN
+	1    1900 4250
+	-1   0    0    1
+$EndComp
+$Comp
+L CONN_01X02 CN3
+U 1 1 54C1676B
+P 4400 3850
+F 0 "CN3" H 4400 4000 50  0000 C CNN
+F 1 "CONN_01X02" V 4500 3850 50  0001 C CNN
+F 2 "HERMESLITE:JUMPER" H 4400 3850 60  0001 C CNN
+F 3 "" H 4400 3850 60  0000 C CNN
+	1    4400 3850
+	1    0    0    1
+$EndComp
+Wire Wire Line
+	2100 3900 2250 3900
+Wire Wire Line
+	2250 3900 2250 4000
+Wire Wire Line
+	2100 4300 2250 4300
+Wire Wire Line
+	2250 4300 2250 4400
 $EndSCHEMATC
