File: hardware/hl/hermeslite.kicad_pcb (KiCad board)
At the start: 2 copper layers, 100 x 80 mm, 37 parts, among them CN1 MagJack, CN10 sata, CN11 RELAYCNT2, CN2 CONN_01X02, CN3 CONN_01X03, CN5 AB2_JACK_3.5MM-3P, CN6 AB2_JACK_3.5MM-3P, CN7 USBBlaster2, CN8 COMPANIONIO, CN9 sata, P1 SMA, P2 SMA, SW1 SW_DIP_4, U1 AD9866BCPZ, U2 KSZ9031RN, U3 FPGA, U4 MCP4716, U5 5P49V5923, U6 ULN2803, U7 TLV62130, X2 38.4MHz

Commit message: More floor and wire planning
Parts:
- added REF**: RF, HERMESLITE:RFCONNECTOR, F.Cu at (186.9, 60.1)
- added REF**: RF, HERMESLITE:RFCONNECTOR, F.Cu at (174.2, 60.1)
- added REF**: RF, HERMESLITE:RFCONNECTOR, F.Cu at (161.5, 60.1)
- CN1: footprint HERMESLITE:MAGJACK -> HERMESLITE:MAGJACK2
- CN11, CN3, CN8, D1, D2, D3, D4: moved to B.Cu
- SW1: value SW_DIP_4 -> SW_DIP_2; footprint HERMESLITE:DIPSW -> HERMESLITE:DIPSW2
- moved D2 27.2 mm to (166.4, 138.9), turned to 180 degrees
- moved D1 24.2 mm to (161.0, 138.9), turned to 180 degrees
- moved D3 23.5 mm to (171.8, 138.9), turned to 180 degrees
- moved D4 21.3 mm to (177.2, 138.9), turned to 180 degrees
- moved U1 13.2 mm to (175.3, 111.4)
- moved P2 5.66 mm to (148.1, 60.1)
- moved CN5 3.80 mm to (131.0, 136.3)
- moved CN6 3.80 mm to (141.6, 136.3)
- moved X2 3.20 mm to (149.3, 76.4), turned to 90 degrees
- moved CN1 3.14 mm to (132.4, 68.6), turned to 180 degrees
- moved P1 2.28 mm to (151.5, 139.6)
- moved U2 1.62 mm to (133.7, 88.3)
- moved SW1 0.51 mm to (121.9, 132.1)
- moved CN10 0.20 mm to (167.1, 131.6)
Connections:
- CN1 pad 12: Net-(C22-Pad1) (its old number) -> Net-(CN1-Pad12)
- CN1 pad 15: Net-(CN1-Pad15) -> GND
- CN1 pad 6: Net-(C26-Pad1) -> Net-(CN1-Pad6)
- CN1 pad 7: Net-(C30-Pad1) -> Net-(CN1-Pad7)
- SW1 pad 1: Net-(R49-Pad1) -> Net-(R44-Pad1)
- SW1 pad 2: Net-(R44-Pad1) -> Net-(R49-Pad1)
- SW1 pad 3: Net-(R38-Pad1) -> GND
- SW1 pad 4: Net-(R34-Pad1) -> GND
- U2 pad 15: Net-(CN1-Pad13) -> Net-(CN1-Pad12)
- U2 pad 17: Net-(CN1-Pad15) -> Net-(CN1-Pad14)
- U2 pad 2: Net-(CN1-Pad11) -> Net-(CN1-Pad2)
- U2 pad 3: Net-(CN1-Pad10) -> Net-(CN1-Pad3)
- U2 pad 7: Net-(CN1-Pad3) -> Net-(CN1-Pad6)
- U2 pad 8: Net-(CN1-Pad2) -> Net-(CN1-Pad7)
- U3 pad 10: (no net) -> Net-(R32-Pad1)
- U3 pad 100: (no net) -> Net-(R11-Pad2)
- U3 pad 101: (no net) -> /Ethernet/RXD0
- U3 pad 102: (no net) -> /Ethernet/RXD1
- U3 pad 105: (no net) -> /Ethernet/RXD2
- U3 pad 106: (no net) -> /Ethernet/RXD3
- U3 pad 11: (no net) -> Net-(R36-Pad1)
- U3 pad 110: (no net) -> Net-(U2-Pad25)
- U3 pad 111: (no net) -> Net-(U2-Pad24)
- U3 pad 116: (no net) -> Net-(CN8-Pad1)
- U3 pad 117: (no net) -> /Ethernet/TXD3
- U3 pad 118: (no net) -> /Ethernet/TXD2
- U3 pad 119: (no net) -> /Ethernet/TXD1
- U3 pad 12: (no net) -> Net-(R33-Pad1)
- U3 pad 120: (no net) -> /Ethernet/TXD0
- U3 pad 123: (no net) -> Net-(U3-Pad123)
- U3 pad 124: Net-(R44-Pad1) -> Net-(R38-Pad1)
- U3 pad 125: Net-(R38-Pad1) -> Net-(R34-Pad1)
- U3 pad 126: (no net) -> Net-(U3-Pad126)
- U3 pad 127: (no net) -> Net-(U3-Pad127)
- U3 pad 128: Net-(R34-Pad1) -> Net-(R44-Pad1)
- U3 pad 129: (no net) -> Net-(U3-Pad129)
- U3 pad 13: (no net) -> Net-(R37-Pad1)
- U3 pad 131: (no net) -> Net-(U3-Pad131)
- U3 pad 132: (no net) -> Net-(U3-Pad132)
- U3 pad 133: (no net) -> Net-(CN8-Pad4)
- U3 pad 135: (no net) -> Net-(CN8-Pad5)
- U3 pad 14: (no net) -> Net-(D1-Pad1)
- U3 pad 140: (no net) -> Net-(CN8-Pad6)
- U3 pad 141: (no net) -> Net-(R49-Pad1)
- U3 pad 20: (no net) -> Net-(D2-Pad1)
- U3 pad 21: (no net) -> Net-(U1-Pad30)
- U3 pad 22: (no net) -> Net-(U1-Pad29)
- U3 pad 23: (no net) -> Net-(U1-Pad28)
- U3 pad 25: (no net) -> Net-(U1-Pad27)
- U3 pad 26: (no net) -> Net-(U1-Pad26)
- U3 pad 27: (no net) -> Net-(U1-Pad25)
- U3 pad 28: (no net) -> Net-(C127-Pad1)
- U3 pad 29: (no net) -> Net-(U1-Pad24)
- U3 pad 30: (no net) -> Net-(U1-Pad23)
- U3 pad 32: (no net) -> Net-(U1-Pad22)
- U3 pad 33: (no net) -> Net-(JP2-Pad2)
- U3 pad 38: (no net) -> Net-(CN10-Pad6)
- U3 pad 39: (no net) -> Net-(CN10-Pad5)
- U3 pad 40: (no net) -> Net-(CN10-Pad3)
- U3 pad 41: (no net) -> Net-(CN10-Pad2)
- U3 pad 42: (no net) -> Net-(CN9-Pad6)
- U3 pad 43: (no net) -> Net-(CN9-Pad5)
- U3 pad 44: (no net) -> Net-(U1-Pad21)
- U3 pad 46: (no net) -> Net-(CN9-Pad3)
- U3 pad 49: (no net) -> Net-(CN9-Pad2)
- U3 pad 50: (no net) -> Net-(U1-Pad20)
- U3 pad 51: (no net) -> Net-(U1-Pad19)
- U3 pad 52: (no net) -> Net-(U1-Pad16)
- U3 pad 53: (no net) -> Net-(U1-Pad15)
- U3 pad 55: (no net) -> Net-(U1-Pad14)
- U3 pad 57: (no net) -> Net-(U3-Pad57)
- U3 pad 58: (no net) -> Net-(U3-Pad58)
- U3 pad 60: (no net) -> Net-(U1-Pad13)
- U3 pad 61: (no net) -> Net-(U1-Pad12)
- U3 pad 62: (no net) -> Net-(U3-Pad62)
- U3 pad 63: (no net) -> Net-(U1-Pad11)
- U3 pad 64: (no net) -> Net-(U1-Pad10)
- U3 pad 65: (no net) -> Net-(U1-Pad9)
- U3 pad 66: (no net) -> Net-(U1-Pad8)
- U3 pad 69: (no net) -> Net-(U1-Pad7)
- U3 pad 70: (no net) -> Net-(U1-Pad6)
- U3 pad 74: (no net) -> Net-(U1-Pad5)
- U3 pad 75: (no net) -> Net-(U1-Pad4)
- U3 pad 76: (no net) -> Net-(U1-Pad3)
- U3 pad 77: (no net) -> Net-(U1-Pad2)
- U3 pad 80: (no net) -> Net-(U1-Pad1)
- U3 pad 81: (no net) -> Net-(U1-Pad62)
- U3 pad 82: (no net) -> Net-(U1-Pad54)
- U3 pad 83: (no net) -> Net-(U1-Pad53)
- U3 pad 84: (no net) -> Net-(U3-Pad84)
- U3 pad 85: (no net) -> Net-(U3-Pad85)
- U3 pad 86: (no net) -> Net-(U3-Pad86)
- U3 pad 87: (no net) -> /Clock/CLKSDA
- U3 pad 88: (no net) -> /Clock/CLKSEL
- U3 pad 89: (no net) -> Net-(U1-Pad61)
- U3 pad 90: (no net) -> Net-(U2-Pad42)
- U3 pad 91: (no net) -> /Ethernet/CLK125
- U3 pad 92: (no net) -> Net-(R16-Pad1)
- U3 pad 93: (no net) -> Net-(R17-Pad1)
- U3 pad 96: (no net) -> Net-(U2-Pad36)
- U3 pad 97: (no net) -> Net-(CN8-Pad3)
- U3 pad 98: (no net) -> Net-(CN8-Pad2)
- U3 pad 99: (no net) -> Net-(R18-Pad2)
- U6 pad 1: Net-(U3-Pad~) -> Net-(U3-Pad132)
- U6 pad 2: Net-(U3-Pad~) -> Net-(U3-Pad131)
- U6 pad 3: Net-(U3-Pad~) -> Net-(U3-Pad129)
- U6 pad 4: Net-(U3-Pad~) -> Net-(U3-Pad127)
- U6 pad 5: Net-(U3-Pad~) -> Net-(U3-Pad126)
- U6 pad 6: Net-(U3-Pad~) -> Net-(R34-Pad1)
- U6 pad 7: Net-(U3-Pad~) -> Net-(R38-Pad1)
- U6 pad 8: Net-(U3-Pad~) -> Net-(U3-Pad123)

Commit message: New floorplan
Parts:
- added C130: 75pF, HERMESLITE:SMD-0805, F.Cu at (145.0, 143.9)
- added C131: 150pF, HERMESLITE:SMD-0805, F.Cu at (150.0, 150.1)
- added C132: 160pF, HERMESLITE:SMD-0805, F.Cu at (150.0, 150.1)
- added C133: 100pF, HERMESLITE:SMD-0805, F.Cu at (150.0, 150.1)
- added C134, C135, C136, C140, C143, C146, C147, C148: 0.1uF, HERMESLITE:SMD-0805, F.Cu at (150.0, 150.1)
- added L10, L9: 240nH, HERMESLITE:SMD-0805, F.Cu at (150.0, 150.1)
- added L11, L12, L13, L14: 270nH, HERMESLITE:SMD-0805, F.Cu at (150.0, 150.1)
- added R57, R58, R59, R62: 1K, HERMESLITE:SMD-0805, F.Cu at (150.0, 150.1)
- added R63, R64: 22, HERMESLITE:SMD-0805, F.Cu at (150.0, 150.1)
- added R65: 75, HERMESLITE:SMD-0805, F.Cu at (150.0, 150.1)
- added R66, R67: 330, HERMESLITE:SMD-0805, F.Cu at (150.0, 150.1)
- moved P1 79.9 mm to (141.8, 60.2), turned to 180 degrees
- moved SW1 75.1 mm to (151.1, 62.9)
- moved CN1 62.9 mm to (137.9, 131.3), turned to 0 degrees
- moved CN6 46.5 mm to (188.1, 136.3)
- moved P2 36.3 mm to (111.8, 60.5)
- moved U2 26.8 mm to (138.0, 114.8), turned to 90 degrees
- moved U4 12.8 mm to (140.1, 80.2)
- moved CN11 12.5 mm to (127.8, 63.3)
- moved U3 12.0 mm to (144.9, 96.8), turned to 0 degrees
- moved U6 11.2 mm to (126.5, 73.3)
- moved CN9 10.5 mm to (174.5, 131.6)
- moved CN10 10.4 mm to (156.7, 131.6)
- moved X2 9.90 mm to (139.9, 73.2)
- moved U5 9.73 mm to (147.9, 78.5)
- moved D1 7.90 mm to (153.1, 138.9)
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Connections:
- U3 pad 10: Net-(R32-Pad1) -> (no net)
- U3 pad 100: Net-(R11-Pad2) -> Net-(U1-Pad10)
- U3 pad 101: /Ethernet/RXD0 -> Net-(U1-Pad9)
- U3 pad 102: /Ethernet/RXD1 -> Net-(U1-Pad8)
- U3 pad 105: /Ethernet/RXD2 -> Net-(U1-Pad7)
- U3 pad 106: /Ethernet/RXD3 -> Net-(U1-Pad6)
- U3 pad 11: Net-(R36-Pad1) -> (no net)
- U3 pad 110: Net-(U2-Pad25) -> Net-(U1-Pad5)
- U3 pad 111: Net-(U2-Pad24) -> Net-(U1-Pad4)
- U3 pad 116: Net-(CN8-Pad1) -> (no net)
- U3 pad 117: /Ethernet/TXD3 -> Net-(U1-Pad3)
- U3 pad 118: /Ethernet/TXD2 -> Net-(U1-Pad2)
- U3 pad 119: /Ethernet/TXD1 -> Net-(U1-Pad1)
- U3 pad 120: /Ethernet/TXD0 -> Net-(U1-Pad62)
- U3 pad 123: Net-(U3-Pad123) -> (no net)
- U3 pad 126: Net-(U3-Pad126) -> (no net)
- U3 pad 127: Net-(U3-Pad127) -> (no net)
- U3 pad 129: Net-(U3-Pad129) -> (no net)
- U3 pad 131: Net-(U3-Pad131) -> (no net)
- U3 pad 132: Net-(U3-Pad132) -> (no net)
- U3 pad 133: Net-(CN8-Pad4) -> (no net)
- U3 pad 135: Net-(CN8-Pad5) -> (no net)
- U3 pad 14: Net-(D1-Pad1) -> (no net)
- U3 pad 140: Net-(CN8-Pad6) -> (no net)
- U3 pad 141: Net-(R49-Pad1) -> (no net)
- U3 pad 20: Net-(D2-Pad1) -> (no net)
- U3 pad 21: Net-(U1-Pad30) -> (no net)
- U3 pad 22: Net-(U1-Pad29) -> (no net)
- U3 pad 23: Net-(U1-Pad28) -> (no net)
- U3 pad 25: Net-(U1-Pad27) -> (no net)
- U3 pad 26: Net-(U1-Pad26) -> (no net)
- U3 pad 27: Net-(U1-Pad25) -> Net-(U2-Pad42)
- U3 pad 28: Net-(C127-Pad1) -> /Ethernet/CLK125
- U3 pad 29: Net-(U1-Pad24) -> Net-(R16-Pad1)
- U3 pad 30: Net-(U1-Pad23) -> Net-(R17-Pad1)
- U3 pad 32: Net-(U1-Pad22) -> Net-(U2-Pad36)
- U3 pad 38: Net-(CN10-Pad6) -> Net-(R18-Pad2)
- U3 pad 39: Net-(CN10-Pad5) -> Net-(R11-Pad2)
- U3 pad 40: Net-(CN10-Pad3) -> /Ethernet/RXD0
- U3 pad 41: Net-(CN10-Pad2) -> /Ethernet/RXD1
- U3 pad 42: Net-(CN9-Pad6) -> /Ethernet/RXD2
- U3 pad 43: Net-(CN9-Pad5) -> /Ethernet/RXD3
- U3 pad 44: Net-(U1-Pad21) -> (no net)
- U3 pad 46: Net-(CN9-Pad3) -> Net-(U2-Pad25)
- U3 pad 49: Net-(CN9-Pad2) -> Net-(U2-Pad24)
- U3 pad 50: Net-(U1-Pad20) -> (no net)
- U3 pad 51: Net-(U1-Pad19) -> /Ethernet/TXD3
- U3 pad 52: Net-(U1-Pad16) -> /Ethernet/TXD2
- U3 pad 53: Net-(U1-Pad15) -> /Ethernet/TXD1
- U3 pad 55: Net-(U1-Pad14) -> /Ethernet/TXD0
- U3 pad 57: Net-(U3-Pad57) -> (no net)
- U3 pad 58: Net-(U3-Pad58) -> (no net)
- U3 pad 60: Net-(U1-Pad13) -> Net-(CN10-Pad6)
- U3 pad 61: Net-(U1-Pad12) -> Net-(CN10-Pad5)
- U3 pad 62: Net-(U3-Pad62) -> (no net)
- U3 pad 63: Net-(U1-Pad11) -> Net-(CN10-Pad3)
- U3 pad 64: Net-(U1-Pad10) -> Net-(CN10-Pad2)
- U3 pad 65: Net-(U1-Pad9) -> Net-(CN9-Pad6)
- U3 pad 66: Net-(U1-Pad8) -> Net-(CN9-Pad5)
- U3 pad 69: Net-(U1-Pad7) -> Net-(CN9-Pad3)
- U3 pad 70: Net-(U1-Pad6) -> Net-(CN9-Pad2)
- U3 pad 74: Net-(U1-Pad5) -> (no net)
- U3 pad 75: Net-(U1-Pad4) -> Net-(U1-Pad30)
- U3 pad 76: Net-(U1-Pad3) -> Net-(U1-Pad29)
- U3 pad 77: Net-(U1-Pad2) -> Net-(U1-Pad28)
- U3 pad 80: Net-(U1-Pad1) -> Net-(U1-Pad27)
- U3 pad 81: Net-(U1-Pad62) -> Net-(U1-Pad26)
- U3 pad 82: Net-(U1-Pad54) -> Net-(U1-Pad25)
- U3 pad 83: Net-(U1-Pad53) -> Net-(U1-Pad24)
- U3 pad 84: Net-(U3-Pad84) -> Net-(U1-Pad23)
- U3 pad 85: Net-(U3-Pad85) -> Net-(U1-Pad22)
- U3 pad 86: Net-(U3-Pad86) -> Net-(U1-Pad21)
- U3 pad 87: /Clock/CLKSDA -> Net-(U1-Pad20)
- U3 pad 88: /Clock/CLKSEL -> (no net)
- U3 pad 89: Net-(U1-Pad61) -> (no net)
- U3 pad 90: Net-(U2-Pad42) -> Net-(U1-Pad19)
- U3 pad 91: /Ethernet/CLK125 -> Net-(U1-Pad16)
- U3 pad 92: Net-(R16-Pad1) -> Net-(U1-Pad15)
- U3 pad 93: Net-(R17-Pad1) -> Net-(U1-Pad14)
- U3 pad 96: Net-(U2-Pad36) -> Net-(U1-Pad13)
- U3 pad 97: Net-(CN8-Pad3) -> (no net)
- U3 pad 98: Net-(CN8-Pad2) -> Net-(U1-Pad12)
- U3 pad 99: Net-(R18-Pad2) -> Net-(U1-Pad11)
- U6 pad 1: Net-(U3-Pad132) -> Net-(U3-Pad~)
- U6 pad 2: Net-(U3-Pad131) -> Net-(U3-Pad~)
- U6 pad 3: Net-(U3-Pad129) -> Net-(U3-Pad~)
- U6 pad 4: Net-(U3-Pad127) -> Net-(U3-Pad~)
- U6 pad 5: Net-(U3-Pad126) -> Net-(U3-Pad~)
- U6 pad 8: Net-(U3-Pad123) -> Net-(U3-Pad~)

Commit message: Latest v2 work
Parts:
- removed C130: 75pF, HERMESLITE:SMD-0805
- removed C131: 150pF, HERMESLITE:SMD-0805
- removed C132: 160pF, HERMESLITE:SMD-0805
- removed C133: 100pF, HERMESLITE:SMD-0805
- removed C134, C135, C136, C140, C143, C146, C147, C148: 0.1uF, HERMESLITE:SMD-0805
- removed CN1: MagJack, HERMESLITE:MAGJACK2
- removed CN10, CN9: sata, HERMESLITE:SATA
- removed CN11: RELAYCNT2, HERMESLITE:FIVEBYTWO
- removed CN8: COMPANIONIO, HERMESLITE:FIVEBYTWO
- removed D1: Led_Small, HERMESLITE:LED
- removed the FIDUCIAL at (102.2, 66.2) (x2)
- removed L10, L9: 240nH, HERMESLITE:SMD-0805
- removed L11, L12, L13, L14: 270nH, HERMESLITE:SMD-0805
- removed P1, P2: SMA, HERMESLITE:SMAEDGE
- removed R57, R58, R59, R62: 1K, HERMESLITE:SMD-0805
- removed R63, R64: 22, HERMESLITE:SMD-0805
- removed R65: 75, HERMESLITE:SMD-0805
- removed R66, R67: 330, HERMESLITE:SMD-0805
- removed REF** (x3): RF, HERMESLITE:RFCONNECTOR
- removed SW1: SW_DIP_2, HERMESLITE:DIPSW2
- removed U1: AD9866BCPZ, HERMESLITE:AD9866
- removed U2: KSZ9031RN, HERMESLITE:KSZ9031
- removed U5: 5P49V5923, HERMESLITE:IDTVERSA
- removed U6: ULN2803, HERMESLITE:PSOP-18
- removed U7: TLV62130, HERMESLITE:TLV62130
- removed X2: 38.4MHz, HERMESLITE:MULTIOSC
- added B36: 0.1uF, HERMESLITE:SMD-0603, B.Cu at (90.2, 48.5)
- added B37: 0.1uF, HERMESLITE:SMD-0603, B.Cu at (87.7, 48.5)
- added B38: 0.1uF, HERMESLITE:SMD-0603, B.Cu at (87.7, 65.1)
- added B39: 0.1uF, HERMESLITE:SMD-0603, B.Cu at (90.2, 65.1)
- added B40: 0.1uF, HERMESLITE:SMD-0603, B.Cu at (95.5, 55.9)
- added B41: 0.1uF, HERMESLITE:SMD-0603, B.Cu at (95.5, 57.5)
- added B42: 0.1uF, HERMESLITE:SMD-0603, B.Cu at (95.1, 53.0)
- added B43: 0.1uF, HERMESLITE:SMD-0603, B.Cu at (95.5, 59.2)
- added B44: 0.1uF, HERMESLITE:SMD-0603, B.Cu at (96.7, 53.0)
- added B45: 0.1uF, HERMESLITE:SMD-0603, B.Cu at (95.6, 61.1)
- added B46: 0.1uF, HERMESLITE:SMD-0603, B.Cu at (99.8, 60.3)
- added B47: 0.1uF, HERMESLITE:SMD-0603, B.Cu at (101.5, 60.3)
- added B48: 0.1uF, HERMESLITE:SMD-0603, B.Cu at (103.2, 58.3)
- added B49: 0.1uF, HERMESLITE:SMD-0603, B.Cu at (103.2, 56.6)
- added B50: 0.1uF, HERMESLITE:SMD-0603, B.Cu at (102.1, 53.0)
- added B51: 0.1uF, HERMESLITE:SMD-0603, B.Cu at (97.9, 58.1)
- added B52: 0.1uF, HERMESLITE:SMD-0603, B.Cu at (100.5, 55.4)
- added B53: 0.1uF, HERMESLITE:SMD-0603, B.Cu at (99.9, 53.0)
- added B54: 0.1uF, HERMESLITE:SMD-0603, B.Cu at (98.3, 53.0)
- added C10: DNI, HERMESLITE:SMD-0805, B.Cu at (158.5, 84.6)
- added C11: 2nF, HERMESLITE:SMD-0805, B.Cu at (160.5, 84.7)
- added C12: 22uF, HERMESLITE:SMD-1210, F.Cu at (145.5, 98.9)
- added C13: 10uF, HERMESLITE:SMD-0805, B.Cu at (163.1, 94.0)
- added C14: 10uF, HERMESLITE:SMD-0805, B.Cu at (163.1, 89.9)
- added C15: 47pF, HERMESLITE:SMD-0805, F.Cu at (158.1, 81.2)
- added C16: 47nF, HERMESLITE:SMD-0805, F.Cu at (159.9, 88.5)
- added C17: 22uF, HERMESLITE:SMD-0805, B.Cu at (167.6, 88.4)
- added C18: 22uF, HERMESLITE:SMD-0805, B.Cu at (170.1, 88.5)
- added C19: DNI, HERMESLITE:SMD-0805, F.Cu at (162.5, 104.9)
- added C20: 2nF, HERMESLITE:SMD-0805, F.Cu at (162.5, 102.6)
- added C21: 33pF, HERMESLITE:SMD-0805, F.Cu at (153.5, 103.1)
- added C22: 1uF, HERMESLITE:SMD-0805, F.Cu at (153.0, 97.6)
- added C23: 47nF, HERMESLITE:SMD-0805, F.Cu at (157.7, 97.6)
- added C24: 22uF, HERMESLITE:SMD-0805, B.Cu at (167.7, 96.4)
- added C25: 22uF, HERMESLITE:SMD-0805, B.Cu at (170.1, 96.4)
- added C26: 10nF, HERMESLITE:SMD-0805, F.Cu at (160.5, 84.6)
- added C27: DNI, HERMESLITE:SMD-0805, F.Cu at (147.0, 80.9)
- added C28: 1.5nF, HERMESLITE:SMD-0805, F.Cu at (143.7, 83.9)
- added C29: 10nF, HERMESLITE:SMD-0805, F.Cu at (143.9, 86.6)
- added C30: 150pF, HERMESLITE:SMD-0805, F.Cu at (137.6, 80.8)
- added C31: 47nF, HERMESLITE:SMD-0805, F.Cu at (148.5, 89.0)
- added C32: 22uF, HERMESLITE:SMD-0805, B.Cu at (138.3, 90.7)
- added C33: 22uF, HERMESLITE:SMD-0805, B.Cu at (140.5, 90.9)
- added C34: 22uF, HERMESLITE:SMD-0805, B.Cu at (142.7, 91.0)
- added C35: 10uF, HERMESLITE:SMD-0603, F.Cu at (111.7, 49.2)
- added C36: 15pF, HERMESLITE:SMD-0603, F.Cu at (93.8, 50.5)
- added C37: 15pF, HERMESLITE:SMD-0603, F.Cu at (96.8, 47.8)
- added C38: 10uF, HERMESLITE:SMD-0603, F.Cu at (103.4, 44.9)
- added C39: 10uF, HERMESLITE:SMD-0603, B.Cu at (103.4, 48.3)
- added C40: 10uF, HERMESLITE:SMD-0603, F.Cu at (103.4, 48.3)
- added CL1: SMA, HERMESLITE:SMAEDGE, F.Cu at (202.0, 92.0)
- added CL3: SMA, HERMESLITE:SMAEDGE, F.Cu at (70.0, 128.2)
- added CN4: RFD4d, HERMESLITE:4x1, F.Cu at (71.5, 88.8)
- added D5: Led_Small, HERMESLITE:LED, B.Cu at (71.1, 74.0)
- added F1: 3A@20V, HERMESLITE:FUSE, F.Cu at (137.8, 106.2)
- added FB10: FB, HERMESLITE:SMD-0603, B.Cu at (103.4, 50.0)
- added FB11: FB, HERMESLITE:SMD-0603, F.Cu at (103.4, 50.0)
- added FB9: FB, HERMESLITE:SMD-0603, F.Cu at (103.4, 46.6)
- added J1: JNC, HERMESLITE:SMD-0603, F.Cu at (111.7, 51.2)
- added L1: 6.8uH, HERMESLITE:NRS8030, F.Cu at (165.9, 87.7)
- added L2: 6.8uH, HERMESLITE:NRS8030, F.Cu at (163.8, 97.3)
- added L3: 2.3uH, HERMESLITE:NRS6045, F.Cu at (143.0, 91.3)
- added Q1: DMP3099L, HERMESLITE:SOT23_3, F.Cu at (134.6, 117.9)
- added R10: 10K, HERMESLITE:SMD-0805, B.Cu at (158.1, 81.3)
- added R11: DNI, HERMESLITE:SMD-0805, F.Cu at (184.1, 86.5)
- added R12: 36K, HERMESLITE:SMD-0805, F.Cu at (158.6, 102.6)
- added R13: 45.3K, HERMESLITE:SMD-0805, F.Cu at (155.3, 99.8)
- added R14: 10K, HERMESLITE:SMD-0805, F.Cu at (155.7, 102.9)
- added R15: DNI, HERMESLITE:SMD-0805, F.Cu at (181.5, 97.6)
- added R16: 21K, HERMESLITE:SMD-0805, F.Cu at (155.1, 86.5)
- added R17: 21K, HERMESLITE:SMD-0805, F.Cu at (147.5, 83.9)
- added R18: 10K, HERMESLITE:SMD-0805, F.Cu at (150.2, 83.9)
- added R19: 10K, HERMESLITE:SMD-0805, F.Cu at (150.2, 81.4)
- added R20: 2.2K, HERMESLITE:SMD-0603, B.Cu at (110.8, 55.7)
- added R21: 10K, HERMESLITE:SMD-0603, B.Cu at (106.6, 60.8)
- added R22: 10K, HERMESLITE:SMD-0603, B.Cu at (110.8, 60.8)
- added R23: 10K, HERMESLITE:SMD-0603, B.Cu at (106.6, 59.1)
- added R24: 10K, HERMESLITE:SMD-0603, B.Cu at (110.8, 59.1)
- added R25: 10K, HERMESLITE:SMD-0603, B.Cu at (106.6, 57.4)
- added R26: 2.2K, HERMESLITE:SMD-0603, B.Cu at (106.6, 55.7)
- added R27: 10K, HERMESLITE:SMD-0603, B.Cu at (106.6, 54.0)
- added R28: 10K, HERMESLITE:SMD-0603, B.Cu at (110.8, 57.4)
- added R29: 10K, HERMESLITE:SMD-0603, B.Cu at (110.8, 54.0)
- added R30: 270, HERMESLITE:SMD-0603, F.Cu at (95.6, 63.5)
- added R31: 270, HERMESLITE:SMD-0603, F.Cu at (100.1, 47.9)
- added R32: 1K, HERMESLITE:SMD-0603, B.Cu at (78.2, 66.3)
- added R33: 1K, HERMESLITE:SMD-0603, B.Cu at (78.2, 47.3)
- added R34: 12.1K, HERMESLITE:SMD-0603, B.Cu at (93.8, 49.8)
- added R8: 27K, HERMESLITE:SMD-0805, B.Cu at (159.9, 87.7)
- added R9: 31.6K, HERMESLITE:SMD-0805, F.Cu at (155.8, 83.1)
- added TP1: TEST_1P, HERMESLITE:TP, F.Cu at (158.3, 111.9)
- added TP2: TEST_1P, HERMESLITE:TP, F.Cu at (149.2, 105.8)
- added TP3: TEST_1P, HERMESLITE:TP, F.Cu at (154.4, 106.3)
- added TP4: TEST_1P, HERMESLITE:TP, F.Cu at (160.1, 108.4)
- added X1: 25MHz, HERMESLITE:XTAL, F.Cu at (96.8, 50.4)
- CN2: value CONN_01X02 -> PS
- CN3: value CONN_01X03 -> MagJack; footprint HERMESLITE:COMPANIONPWR -> HERMESLITE:MAGJACK; moved to F.Cu
- CN5, CN6: value AB2_JACK_3.5MM-3P -> RFD4d; footprint HERMESLITE:CWJACK -> HERMESLITE:4x1
- CN7: value USBBlaster2 -> RFD4d; footprint HERMESLITE:USBBLASTER -> HERMESLITE:4x1
- D2, D4: moved to F.Cu
- U3: value FPGA -> TPS65265; footprint HERMESLITE:MAX10 -> HERMESLITE:QFP_32
- U4: value MCP4716 -> KSZ9031RN; footprint HERMESLITE:MCP4716 -> HERMESLITE:KSZ9031
- moved CN2 126.3 mm to (211.3, 53.7), turned to 180 degrees
- moved FIDUCIAL 123.3 mm to (77.0, 41.5) (x2)
- moved FIDUCIAL 120.9 mm to (77.0, 138.5) (x2)
- moved D4 120.0 mm to (71.1, 73.9), turned to 270 degrees
- moved CN6 119.6 mm to (71.5, 109.5), turned to 270 degrees
- moved D3 117.2 mm to (71.1, 69.3), turned to 90 degrees
- moved D2 112.3 mm to (71.1, 69.3), turned to 270 degrees
- moved FIDUCIAL 110.9 mm to (213.0, 138.5) (x2)
- moved CN3 67.2 mm to (81.1, 56.8)
- moved CN5 63.9 mm to (71.5, 99.0), turned to 270 degrees
- moved U4 47.0 mm to (99.3, 56.8)
- moved CN7 39.5 mm to (71.5, 78.6), turned to 270 degrees
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Connections:
- CN3 pad 1: Net-(CN2-Pad1) -> Net-(B38-Pad1)
- CN3 pad 2: GND -> Net-(CN3-Pad2)
- CN3 pad 3: Net-(C17-Pad1) -> Net-(CN3-Pad3)
- CN5 pad 3: GND -> Net-(CN5-Pad3)
- CN5 pad 4: Net-(CN5-Pad4) -> GND
- CN6 pad 3: GND -> Net-(CN6-Pad3)
- CN6 pad 4: Net-(CN6-Pad4) -> GND
- CN7 pad 2: GND -> Net-(CN7-Pad2)
- CN7 pad 4: VCC -> GND
- U3 pad 1: Net-(C103-Pad1) -> Net-(C22-Pad1)
- U3 pad 10: (no net) -> GND
- U3 pad 11: (no net) -> Net-(C23-Pad1)
- U3 pad 12: Net-(C27-Pad1) -> Net-(C12-Pad1)
- U3 pad 13: Net-(C129-Pad1) -> Net-(C12-Pad1)
- U3 pad 14: (no net) -> Net-(C16-Pad1)
- U3 pad 15: Net-(CN7-Pad8) -> GND
- U3 pad 16: Net-(CN7-Pad5) -> Net-(C16-Pad2)
- U3 pad 17: Net-(CN7-Pad1) -> Net-(C26-Pad1)
- U3 pad 18: Net-(CN7-Pad9) -> Net-(C10-Pad2)
- U3 pad 19: Net-(CN7-Pad3) -> Net-(C15-Pad1)
- U3 pad 2: Net-(C100-Pad1) -> Net-(R11-Pad1)
- U3 pad 20: (no net) -> Net-(R16-Pad2)
- U3 pad 21: (no net) -> GND
- U3 pad 22: (no net) -> Net-(C30-Pad1)
- U3 pad 23: (no net) -> Net-(C27-Pad2)
- U3 pad 24: Net-(C101-Pad1) -> Net-(C29-Pad1)
- U3 pad 25: (no net) -> Net-(C31-Pad2)
- U3 pad 26: (no net) -> GND
- U3 pad 27: Net-(U2-Pad42) -> GND
- U3 pad 28: /Ethernet/CLK125 -> Net-(C31-Pad1)
- U3 pad 29: Net-(R16-Pad1) -> Net-(C31-Pad1)
- U3 pad 3: GND -> Net-(TP1-Pad1)
- U3 pad 30: Net-(R17-Pad1) -> Net-(C12-Pad1)
- U3 pad 31: Net-(C101-Pad1) -> Net-(C12-Pad1)
- U3 pad 33: Net-(JP2-Pad2) -> GND
- U3 pad 4: GND -> Net-(TP2-Pad1)
- U3 pad 5: Net-(C100-Pad1) -> Net-(TP3-Pad1)
- U3 pad 6: (no net) -> Net-(C21-Pad1)
- U3 pad 7: (no net) -> Net-(C19-Pad2)
- U3 pad 8: (no net) -> Net-(TP4-Pad1)
- U3 pad 9: Net-(C101-Pad1) -> Net-(C23-Pad2)
- U4 pad 1: Net-(R21-Pad2) -> Net-(B42-Pad1)
- U4 pad 2: GND -> Net-(CN3-Pad11)
- U4 pad 3: Net-(C62-Pad1) -> Net-(CN3-Pad10)
- U4 pad 4: /Clock/CLKSDA -> Net-(B40-Pad1)
- U4 pad 5: /Clock/CLKSEL -> Net-(CN3-Pad5)
- U4 pad 6: Net-(R19-Pad2) -> Net-(CN3-Pad4)
Routing:
- net Net-(CN3-Pad17): track 0.00 -> 45.2 mm, vias 0 -> 1
- net GND: track 0.00 -> 37.0 mm, vias 0 -> 2
- net Net-(CN3-Pad13): track 0.00 -> 35.4 mm
- net Net-(CN3-Pad14): track 0.00 -> 27.4 mm, vias 0 -> 1
- net Net-(CN3-Pad16): track 0.00 -> 27.2 mm
- net Net-(B40-Pad1): track 0.00 -> 25.9 mm, vias 0 -> 4
- net Net-(B42-Pad1): track 0.00 -> 25.6 mm, vias 0 -> 4
- net +1V2: track 0.00 -> 24.6 mm, vias 0 -> 6
- net Veth: track 0.00 -> 24.2 mm, vias 0 -> 4
- net Net-(B54-Pad1): track 0.00 -> 10.9 mm, vias 0 -> 2
- net Net-(CN3-Pad5): track 0.00 -> 9.97 mm
- net Net-(CN3-Pad2): track 0.00 -> 9.46 mm
- net Net-(CN3-Pad4): track 0.00 -> 8.44 mm
- net Net-(CN3-Pad3): track 0.00 -> 8.43 mm
- net Net-(C36-Pad2): track 0.00 -> 6.77 mm
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Other:
- board size 100 x 80 mm -> 150 x 100 mm
- copper layers 2 -> 4
- net class Default: trace_width 0.25 -> 0.2; via_drill 0.4 -> 0.3

Commit message: Before Power Supply Change
Parts:
- added B1: 0.1uF, HERMESLITE:SMD-0603, F.Cu at (123.5, 84.8)
- added B10: 0.1uF, HERMESLITE:SMD-0603, B.Cu at (96.7, 86.7)
- added B11: 0.1uF, HERMESLITE:SMD-0603, B.Cu at (118.2, 69.0)
- added B12: 0.1uF, HERMESLITE:SMD-0603, B.Cu at (102.8, 89.0)
- added B13: 0.1uF, HERMESLITE:SMD-0603, B.Cu at (104.5, 89.0)
- added B14: 0.1uF, HERMESLITE:SMD-0603, B.Cu at (116.2, 85.0)
- added B15: 0.1uF, HERMESLITE:SMD-0603, B.Cu at (116.3, 73.0)
- added B16: 0.1uF, HERMESLITE:SMD-0603, B.Cu at (116.2, 69.7)
- added B17: 0.1uF, HERMESLITE:SMD-0603, B.Cu at (115.5, 66.8)
- added B18: 0.1uF, HERMESLITE:SMD-0603, B.Cu at (104.7, 68.8)
- added B19: 0.1uF, HERMESLITE:SMD-0603, B.Cu at (111.2, 68.8)
- added B2: 0.1uF, HERMESLITE:SMD-0603, B.Cu at (96.7, 67.7)
- added B20: 0.1uF, HERMESLITE:SMD-0603, B.Cu at (100.2, 68.7)
- added B21: 0.1uF, HERMESLITE:SMD-0603, B.Cu at (96.0, 74.2)
- added B22: 0.1uF, HERMESLITE:SMD-0603, B.Cu at (96.2, 71.3)
- added B23: 0.1uF, HERMESLITE:SMD-0603, B.Cu at (98.0, 82.2)
- added B24: 0.1uF, HERMESLITE:SMD-0603, B.Cu at (102.3, 87.0)
- added B25: 0.1uF, HERMESLITE:SMD-0603, B.Cu at (105.7, 87.0)
- added B26: 0.1uF, HERMESLITE:SMD-0603, B.Cu at (110.2, 87.0)
- added B27: 0.1uF, HERMESLITE:SMD-0603, B.Cu at (113.5, 87.0)
- added B28: 0.1uF, HERMESLITE:SMD-0603, B.Cu at (98.0, 79.7)
- added B29: 0.1uF, HERMESLITE:SMD-0603, B.Cu at (98.2, 72.3)
- added B3: 0.1uF, HERMESLITE:SMD-0603, B.Cu at (118.2, 87.2)
- added B30: 0.1uF, HERMESLITE:SMD-0603, B.Cu at (105.8, 66.8)
- added B31: 0.1uF, HERMESLITE:SMD-0603, B.Cu at (102.5, 66.8)
- added B32: 0.1uF, HERMESLITE:SMD-0603, B.Cu at (113.8, 66.8)
- added B33: 0.1uF, HERMESLITE:SMD-0603, B.Cu at (110.2, 66.8)
- added B34: 0.1uF, HERMESLITE:SMD-0603, B.Cu at (118.2, 74.3)
- added B35: 0.1uF, HERMESLITE:SMD-0603, B.Cu at (116.2, 78.2)
- added B4: 0.1uF, HERMESLITE:SMD-0603, B.Cu at (96.5, 88.8)
- added B5: 0.1uF, HERMESLITE:SMD-0603, B.Cu at (117.8, 67.0)
- added B6: 0.1uF, HERMESLITE:SMD-0603, B.Cu at (109.0, 88.8)
- added B7: 0.1uF, HERMESLITE:SMD-0603, B.Cu at (114.3, 89.0)
- added B8: 0.1uF, HERMESLITE:SMD-0603, B.Cu at (96.2, 69.7)
- added B9: 0.1uF, HERMESLITE:SMD-0603, B.Cu at (118.2, 85.7)
- added CN1: USBBlaster2, HERMESLITE:USBBLASTER, F.Cu at (129.2, 79.8)
- added R1: 33, HERMESLITE:SMD-0603, B.Cu at (122.2, 79.0)
- added R2: 10K, HERMESLITE:SMD-0603, B.Cu at (132.8, 79.8)
- added R3: 10K, HERMESLITE:SMD-0603, B.Cu at (128.0, 87.7)
- added R4: 10K, HERMESLITE:SMD-0603, B.Cu at (124.7, 75.8)
- added R5: 10K, HERMESLITE:SMD-0603, B.Cu at (99.7, 78.2)
- added R6: 10K, HERMESLITE:SMD-0603, B.Cu at (115.0, 81.0)
- added R7: 10K, HERMESLITE:SMD-0603, B.Cu at (115.7, 82.8)
- added U1: EEPROM, HERMESLITE:SOIC-8, B.Cu at (123.8, 83.8)
- added U2: FPGA, HERMESLITE:CYCLONEIV, F.Cu at (107.2, 77.8)
- C10, C11, C13, C14, C17, C18, C24, C25, C32, C33, C34, R10, R8: moved to F.Cu
- moved Q1 77.1 mm to (185.3, 59.9)
- moved F1 66.3 mm to (185.3, 59.9)
- moved TP1 58.6 mm to (185.3, 59.9)
- moved TP2 58.4 mm to (185.3, 59.9)
- moved C32 56.2 mm to (185.3, 59.9), turned to 0 degrees
- moved TP3 55.8 mm to (185.3, 59.9)
- moved C12 55.7 mm to (185.3, 59.9), turned to 0 degrees
- moved TP4 54.7 mm to (185.3, 59.9)
- moved C33 54.5 mm to (185.3, 59.9), turned to 0 degrees
- moved C21 53.7 mm to (185.3, 59.9), turned to 0 degrees
- moved C34 52.8 mm to (185.3, 59.9), turned to 0 degrees
- moved L3 52.7 mm to (185.3, 59.9), turned to 0 degrees
- moved R14 52.2 mm to (185.3, 59.9), turned to 0 degrees
- moved C30 52.1 mm to (185.3, 59.9), turned to 0 degrees
- moved C19 50.5 mm to (185.3, 59.9), turned to 0 degrees
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Routing:
- net (no net): track 0.00 -> 121.4 mm
- net GND: track 37.0 -> 115.8 mm, vias 2 -> 45
- net +1V2: track 24.6 -> 53.3 mm, vias 6 -> 20
- net Net-(CN1-Pad5): track 0.00 -> 16.1 mm
- net +3V3: track 0.00 -> 14.7 mm, vias 0 -> 3
- net Net-(U1-Pad6): track 0.00 -> 14.3 mm, vias 0 -> 1
- net Net-(CN1-Pad1): track 0.00 -> 13.8 mm, vias 0 -> 1
- net Net-(U1-Pad5): track 0.00 -> 13.5 mm, vias 0 -> 1
- net Net-(CN1-Pad9): track 0.00 -> 12.0 mm
- net Net-(CN1-Pad3): track 0.00 -> 9.92 mm
- net Net-(U1-Pad1): track 0.00 -> 7.86 mm, vias 0 -> 1
- net Net-(R1-Pad2): track 0.00 -> 6.63 mm, vias 0 -> 1
- net Vb7: track 0.00 -> 4.20 mm, vias 0 -> 2
- net Net-(R5-Pad1): track 0.00 -> 4.03 mm, vias 0 -> 1
- net Vb8: track 0.00 -> 3.97 mm, vias 0 -> 2
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Other:
- net class Default: clearance 0.2 -> 0.19
- rule trace_clearance: 0.2 -> 0.19
