File: hardware/hl/hermeslite.kicad_pcb (KiCad board)
At the start: 4 copper layers, 150 x 100 mm, 160 parts, among them CN1 USBBlaster2, CN2 PS, CN3 MagJack, CN4 RFD4d, CN5 RFD4d, CN6 RFD4d, CN7 RFD4d, J1 JNC, Q1 DMP3099L, U1 EEPROM, U2 FPGA, U3 TPS65265, U4 KSZ9031RN, X1 25MHz

Commit message: More PCB layout
Parts:
- removed C10, C19, C27, R11, R15: DNI, HERMESLITE:SMD-0805
- removed C11, C20: 2nF, HERMESLITE:SMD-0805
- removed C12: 22uF, HERMESLITE:SMD-1210
- removed C13, C14: 10uF, HERMESLITE:SMD-0805
- removed C15: 47pF, HERMESLITE:SMD-0805
- removed C16, C23, C31: 47nF, HERMESLITE:SMD-0805
- removed C17, C18, C24, C25, C32, C33, C34: 22uF, HERMESLITE:SMD-0805
- removed C21: 33pF, HERMESLITE:SMD-0805
- removed C22: 1uF, HERMESLITE:SMD-0805
- removed C26, C29: 10nF, HERMESLITE:SMD-0805
- removed C28: 1.5nF, HERMESLITE:SMD-0805
- removed C30: 150pF, HERMESLITE:SMD-0805
- removed CN6, CN7: RFD4d, HERMESLITE:4x1
- removed L1, L2: 6.8uH, HERMESLITE:NRS8030
- removed L3: 2.3uH, HERMESLITE:NRS6045
- removed R10, R14, R18, R19: 10K, HERMESLITE:SMD-0805
- removed R12: 36K, HERMESLITE:SMD-0805
- removed R13: 45.3K, HERMESLITE:SMD-0805
- removed R16, R17: 21K, HERMESLITE:SMD-0805
- removed R8: 27K, HERMESLITE:SMD-0805
- removed R9: 31.6K, HERMESLITE:SMD-0805
- removed TP1, TP2, TP3, TP4: TEST_1P, HERMESLITE:TP
- removed U3: TPS65265, HERMESLITE:QFP_32
- added C1: 10uF, HERMESLITE:SMD-0603, B.Cu at (93.5, 69.6)
- added C2: 10uF, HERMESLITE:SMD-0603, B.Cu at (115.5, 82.2)
- added C3: 10uF, HERMESLITE:SMD-0603, B.Cu at (98.2, 86.6)
- added C4: 10uF, HERMESLITE:SMD-0603, B.Cu at (120.0, 66.6)
- added C5: 100uF, HERMESLITE:SMD-1210, B.Cu at (108.0, 72.8)
- added C6: 10uF, HERMESLITE:SMD-0603, B.Cu at (111.3, 85.0)
- added C7: 10uF, HERMESLITE:SMD-0603, B.Cu at (112.9, 70.8)
- added C8: 10uF, HERMESLITE:SMD-0603, B.Cu at (103.0, 71.7)
- added C9: 10uF, HERMESLITE:SMD-0603, B.Cu at (104.7, 83.7)
- added DB22: RFD4d, HERMESLITE:4x1, F.Cu at (81.4, 105.3)
- added DB7: RFD4d, HERMESLITE:4x1, F.Cu at (81.0, 69.5)
- added FB1: FB, HERMESLITE:SMD-0603, B.Cu at (96.6, 65.9)
- added FB2: FB, HERMESLITE:SMD-0603, B.Cu at (118.8, 89.3)
- added FB3: FB, HERMESLITE:SMD-0603, B.Cu at (99.2, 88.7)
- added FB4: FB, HERMESLITE:SMD-0603, B.Cu at (117.2, 64.8)
- added FB5: FB, HERMESLITE:SMD-0603, B.Cu at (94.4, 67.5)
- added FB6: FB, HERMESLITE:SMD-0603, B.Cu at (113.0, 82.7)
- added FB7: FB, HERMESLITE:SMD-0603, B.Cu at (97.7, 84.5)
- added FB8: FB, HERMESLITE:SMD-0603, B.Cu at (121.7, 66.6)
- CN4, CN5: value RFD4d -> IO8; footprint HERMESLITE:4x1 -> HERMESLITE:IO
- moved CL1 131.7 mm to (70.1, 123.7), turned to 270 degrees
- moved D3 46.2 mm to (70.9, 115.5)
- moved D4 41.6 mm to (70.9, 115.5)
- moved D2 41.1 mm to (70.9, 110.4)
- moved D5 36.4 mm to (70.9, 110.4)
- moved CL3 25.7 mm to (70.1, 102.5)
- moved Q1 21.1 mm to (203.3, 48.8)
- moved CN4 14.4 mm to (72.7, 74.5)
- moved F1 14.1 mm to (196.1, 50.8)
- moved CN5 9.38 mm to (72.7, 89.7)
- moved R7 4.32 mm to (112.8, 79.5), turned to 90 degrees
- moved R6 1.64 mm to (114.5, 79.5), turned to 90 degrees
- moved B10 0.07 mm to (96.6, 86.6)
- moved B2 0.07 mm to (96.6, 67.6)
- moved B8 0.07 mm to (96.1, 69.6)
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Connections:
- net Vb5 renamed Vlvds
- B12 pad 1: Vb7 -> +3V3
- B13 pad 1: Vb7 -> +3V3
- B28 pad 1: Vb6 -> +3V3
- B30 pad 1: Vb4 -> Veth
- B31 pad 1: Vb4 -> Veth
- B32 pad 1: Vb3 -> Veth
- B33 pad 1: Vb3 -> Veth
- B34 pad 1: Vb2 -> +3V3
- B6 pad 1: Vb8 -> +3V3
- B7 pad 1: Vb8 -> +3V3
- CN4 pad 1: Net-(CN4-Pad1) -> GND
- CN4 pad 4: GND -> Net-(CN4-Pad4)
- CN5 pad 1: Net-(CN5-Pad1) -> GND
- CN5 pad 4: GND -> Net-(CN5-Pad4)
- R5 pad 2: Vb6 -> +3V3
- U2 pad 10: (no net) -> Net-(U2-Pad10)
- U2 pad 105: (no net) -> Net-(U2-Pad105)
- U2 pad 106: (no net) -> Net-(U2-Pad106)
- U2 pad 110: (no net) -> Net-(U2-Pad110)
- U2 pad 111: (no net) -> Net-(U2-Pad111)
- U2 pad 112: (no net) -> Net-(U2-Pad112)
- U2 pad 113: (no net) -> Net-(U2-Pad113)
- U2 pad 114: (no net) -> Net-(U2-Pad114)
- U2 pad 115: (no net) -> Net-(U2-Pad115)
- U2 pad 117: Vb7 -> +3V3
- U2 pad 119: (no net) -> Net-(U2-Pad119)
- U2 pad 120: (no net) -> Net-(U2-Pad120)
- U2 pad 121: (no net) -> Net-(U2-Pad121)
- U2 pad 122: Vb7 -> +3V3
- U2 pad 125: (no net) -> Net-(U2-Pad125)
- U2 pad 126: (no net) -> Net-(U2-Pad126)
- U2 pad 127: (no net) -> Net-(U2-Pad127)
- U2 pad 128: (no net) -> Net-(U2-Pad128)
- U2 pad 129: (no net) -> Net-(U2-Pad129)
- U2 pad 130: Vb8 -> +3V3
- U2 pad 132: (no net) -> Net-(U2-Pad132)
- U2 pad 133: (no net) -> Net-(U2-Pad133)
- U2 pad 135: (no net) -> Net-(U2-Pad135)
- U2 pad 136: (no net) -> Net-(U2-Pad136)
- U2 pad 137: (no net) -> Net-(U2-Pad137)
- U2 pad 139: Vb8 -> +3V3
- U2 pad 141: (no net) -> Net-(U2-Pad141)
- U2 pad 142: (no net) -> Net-(U2-Pad142)
- U2 pad 143: (no net) -> Net-(U2-Pad143)
- U2 pad 144: (no net) -> Net-(U2-Pad144)
- U2 pad 26: Vb2 -> +3V3
- U2 pad 40: Vb3 -> Veth
- U2 pad 47: Vb3 -> Veth
- U2 pad 49: (no net) -> Net-(J1-Pad1)
- U2 pad 50: (no net) -> Net-(R26-Pad2)
- U2 pad 51: (no net) -> Net-(U2-Pad51)
- U2 pad 52: (no net) -> Net-(R27-Pad1)
- U2 pad 53: (no net) -> Net-(R28-Pad1)
- U2 pad 54: (no net) -> Net-(R25-Pad2)
- U2 pad 55: (no net) -> /Ethernet/RXD0
- U2 pad 56: Vb4 -> Veth
- U2 pad 58: (no net) -> /Ethernet/RXD1
- U2 pad 59: (no net) -> /Ethernet/RXD2
- U2 pad 60: (no net) -> /Ethernet/RXD3
- U2 pad 62: Vb4 -> Veth
- U2 pad 64: (no net) -> Net-(U2-Pad64)
- U2 pad 65: (no net) -> Net-(U2-Pad65)
- U2 pad 66: (no net) -> /Ethernet/TXD3
- U2 pad 67: (no net) -> /Ethernet/TXD2
- U2 pad 68: (no net) -> /Ethernet/TXD1
- U2 pad 69: (no net) -> /Ethernet/TXD0
- U2 pad 7: (no net) -> Net-(U2-Pad7)
- U2 pad 71: (no net) -> Net-(DB7-Pad2)
- U2 pad 72: (no net) -> Net-(DB7-Pad3)
- U2 pad 76: (no net) -> Net-(C71-Pad1)
- U2 pad 77: (no net) -> Net-(C72-Pad1)
- U2 pad 80: (no net) -> Net-(C73-Pad1)
- U2 pad 83: (no net) -> Net-(C74-Pad1)
- U2 pad 85: (no net) -> Net-(D5-Pad1)
- U2 pad 86: (no net) -> Net-(C75-Pad1)
- U2 pad 87: (no net) -> Net-(C76-Pad1)
- U2 pad 88: (no net) -> Net-(C77-Pad1)
- U2 pad 89: (no net) -> Net-(C78-Pad1)
- U2 pad 90: (no net) -> Net-(B65-Pad2)
- U2 pad 91: (no net) -> Net-(B112-Pad2)
- U2 pad 93: Vb6 -> +3V3
- U2 pad 98: (no net) -> Net-(D3-Pad1)
- U2 pad 99: (no net) -> Net-(D4-Pad1)
- U4 pad 24: Net-(U2-Pad~) -> Net-(U2-Pad65)
- U4 pad 25: Net-(U2-Pad~) -> Net-(U2-Pad64)
- U4 pad 36: Net-(U2-Pad~) -> Net-(U2-Pad51)
Routing:
- net +3V3: track 14.7 -> 32.1 mm, vias 3 -> 9
- net Veth: track 24.8 -> 32.6 mm, vias 4 -> 8
- net Net-(B9-Pad1): track 1.77 -> 8.54 mm
- net Net-(R7-Pad1): track 1.88 -> 6.44 mm
- net Vb7: track 4.20 -> 0.00 mm, vias 2 -> 0
- net Vb8: track 3.97 -> 0.00 mm, vias 2 -> 0
- net Vb4: track 3.95 -> 0.00 mm, vias 2 -> 0
- net Vb6: track 3.78 -> 0.00 mm, vias 1 -> 0
- net Vb3: track 3.77 -> 0.00 mm, vias 2 -> 0
- net Net-(B8-Pad1): track 1.82 -> 3.94 mm
- net Vb2: track 1.98 -> 0.00 mm, vias 1 -> 0
- net Net-(B3-Pad1): track 1.84 -> 3.25 mm
- net GND: track 115.8 -> 115.1 mm, vias 45 -> 46
- net Net-(R6-Pad1): track 3.12 -> 3.74 mm

Commit message: Update, more layout
Parts:
- added B112: 0.1uF, HERMESLITE:SMD-0603, F.Cu at (80.2, 100.0)
- added B113: 0.1uF, HERMESLITE:SMD-0603, B.Cu at (93.6, 130.5)
- added B114: 0.1uF, HERMESLITE:SMD-0603, B.Cu at (91.6, 126.8)
- added B115: 0.1uF, HERMESLITE:SMD-0603, B.Cu at (88.9, 129.6)
- added B55: 0.1uF, HERMESLITE:SMD-0603, B.Cu at (81.8, 125.7)
- added B56: 0.1uF, HERMESLITE:SMD-0603, B.Cu at (85.4, 123.6)
- added B57: 0.1uF, HERMESLITE:SMD-0603, F.Cu at (86.7, 130.1)
- added B58: 0.1uF, HERMESLITE:SMD-0603, F.Cu at (81.7, 164.9)
- added B59: 0.1uF, HERMESLITE:SMD-0603, B.Cu at (95.2, 126.9)
- added B60: 0.1uF, HERMESLITE:SMD-0603, B.Cu at (91.6, 124.1)
- added B61: 0.1uF, HERMESLITE:SMD-0603, B.Cu at (89.7, 126.8)
- added B62: 0.1uF, HERMESLITE:SMD-0603, B.Cu at (91.5, 131.7)
- added B63: 0.1uF, HERMESLITE:SMD-0603, F.Cu at (87.6, 132.2)
- added B64: 0.1uF, HERMESLITE:SMD-0603, B.Cu at (92.6, 121.2)
- added B65: 0.1uF, HERMESLITE:SMD-0603, F.Cu at (80.2, 102.6)
- added C10: 1uF, HERMESLITE:SMD-0603, F.Cu at (82.4, 103.2)
- added C11: 1uF, HERMESLITE:SMD-0603, F.Cu at (82.4, 99.4)
- added C12: 10uF, HERMESLITE:SMD-0603, B.Cu at (93.2, 126.8)
- added C41: 10uF, HERMESLITE:SMD-0603, B.Cu at (87.3, 123.1)
- added C42: DNI, HERMESLITE:SMD-0603, F.Cu at (85.0, 132.2)
- added C44: 10uF, HERMESLITE:SMD-0603, B.Cu at (89.9, 131.7)
- added C45: 10uF, HERMESLITE:SMD-0603, B.Cu at (94.9, 121.2)
- added C71: 1uF, HERMESLITE:SMD-0603, F.Cu at (79.5, 69.8)
- added C72: 1uF, HERMESLITE:SMD-0603, F.Cu at (79.5, 72.5)
- added C73: 1uF, HERMESLITE:SMD-0603, F.Cu at (79.5, 75.1)
- added C74: 1uF, HERMESLITE:SMD-0603, F.Cu at (79.5, 77.8)
- added C75: 1uF, HERMESLITE:SMD-0603, F.Cu at (79.5, 85.0)
- added C76: 1uF, HERMESLITE:SMD-0603, F.Cu at (79.5, 87.7)
- added C77: 1uF, HERMESLITE:SMD-0603, F.Cu at (79.5, 90.3)
- added C78: 1uF, HERMESLITE:SMD-0603, F.Cu at (79.5, 93.0)
- added DB1: RFD4d, HERMESLITE:4x1, F.Cu at (89.2, 160.1)
- added FB12: FB, HERMESLITE:SMD-0603, B.Cu at (89.0, 123.1)
- added FB13: FB, HERMESLITE:SMD-0603, B.Cu at (88.2, 131.7)
- added FB23: FB, HERMESLITE:SMD-0603, B.Cu at (87.4, 126.3)
- added FB24: FB, HERMESLITE:SMD-0603, B.Cu at (93.2, 124.1)
- added FB25: FB, HERMESLITE:SMD-0603, B.Cu at (96.4, 124.1)
- added FB26: FB, HERMESLITE:SMD-0603, B.Cu at (94.8, 124.1)
- added J13: JNO, HERMESLITE:SMD-0603, B.Cu at (80.7, 73.8)
- added J14: JNC, HERMESLITE:SMD-0603, F.Cu at (77.3, 73.8)
- added J17: JNO, HERMESLITE:SMD-0603, B.Cu at (80.7, 89.0)
- added J18: JNC, HERMESLITE:SMD-0603, F.Cu at (77.3, 89.0)
- added J3: JNO, HERMESLITE:SMD-0603, B.Cu at (82.6, 123.6)
- added J4: JNO, HERMESLITE:SMD-0603, F.Cu at (86.3, 124.7)
- added R10: 2.2, HERMESLITE:SMD-0603, B.Cu at (87.4, 128.0)
- added R35: 3.3K, HERMESLITE:SMD-0603, B.Cu at (84.0, 127.8)
- added R36: DNI, HERMESLITE:SMD-0603, B.Cu at (80.9, 123.6)
- added R37: 10K, HERMESLITE:SMD-0603, B.Cu at (84.0, 130.5)
- added R38: DNI, HERMESLITE:SMD-0603, F.Cu at (79.8, 123.2)
- added R39: 120, HERMESLITE:SMD-0603, F.Cu at (88.0, 124.7)
- added R40: 75, HERMESLITE:SMD-0603, F.Cu at (87.5, 127.4)
- added R41: DNI, HERMESLITE:SMD-0603, F.Cu at (89.7, 123.7)
- added R42: 33, HERMESLITE:SMD-0603, F.Cu at (93.6, 125.7)
- added R43: 4.7K, HERMESLITE:SMD-0603, F.Cu at (80.5, 161.1)
- added R44: 4.7K, HERMESLITE:SMD-0603, F.Cu at (80.8, 158.3)
- added R45: 33, HERMESLITE:SMD-0603, F.Cu at (97.4, 129.1)
- added R71: 330, HERMESLITE:SMD-0603, F.Cu at (76.6, 109.1)
- added R72: 330, HERMESLITE:SMD-0603, B.Cu at (76.6, 116.7)
- added R73: 330, HERMESLITE:SMD-0603, F.Cu at (76.6, 114.2)
- added R74: 330, HERMESLITE:SMD-0603, B.Cu at (76.6, 111.6)
- added R75: 10K, HERMESLITE:SMD-0603, F.Cu at (81.2, 69.8)
- added R76: 10K, HERMESLITE:SMD-0603, F.Cu at (81.2, 72.5)
- added R77: 330, HERMESLITE:SMD-0603, F.Cu at (77.3, 70.3)
- added R78: 330, HERMESLITE:SMD-0603, F.Cu at (77.3, 72.0)
- added R79: 10K, HERMESLITE:SMD-0603, F.Cu at (81.2, 75.1)
- added R8: 10K, HERMESLITE:SMD-0603, F.Cu at (84.1, 103.2)
- added R80: 10K, HERMESLITE:SMD-0603, F.Cu at (81.2, 77.8)
- added R81: 330, HERMESLITE:SMD-0603, F.Cu at (77.3, 75.6)
- added R82: 330, HERMESLITE:SMD-0603, F.Cu at (77.3, 77.3)
- added R83: 10K, HERMESLITE:SMD-0603, F.Cu at (81.2, 85.0)
- added R84: 10K, HERMESLITE:SMD-0603, F.Cu at (81.2, 87.7)
- added R85: 330, HERMESLITE:SMD-0603, F.Cu at (77.3, 85.5)
- added R86: 330, HERMESLITE:SMD-0603, F.Cu at (77.3, 87.2)
- added R87: 10K, HERMESLITE:SMD-0603, F.Cu at (81.2, 90.3)
- added R88: 10K, HERMESLITE:SMD-0603, F.Cu at (81.2, 93.0)
- added R89: 330, HERMESLITE:SMD-0603, F.Cu at (77.3, 90.8)
- added R9: 10K, HERMESLITE:SMD-0603, F.Cu at (84.1, 99.4)
- added R90: 330, HERMESLITE:SMD-0603, F.Cu at (77.3, 92.5)
- added U5: MCP4716, HERMESLITE:MCP4716, B.Cu at (81.4, 128.7)
- added U6: 5P49V5923, HERMESLITE:IDTVERSA, F.Cu at (91.2, 129.3)
- added X2: 38.4MHz, HERMESLITE:MULTIOSC, F.Cu at (82.1, 127.7)
- moved DB22 4.00 mm to (77.4, 105.1)
- moved DB7 2.65 mm to (83.6, 69.0)
Connections:
- J1 pad 2: (no net) -> Net-(J1-Pad2)
- U2 pad 100: (no net) -> Net-(D4-Pad1)
- U2 pad 49: Net-(J1-Pad1) -> Net-(J1-Pad2)
- U2 pad 98: Net-(D3-Pad1) -> Net-(D2-Pad1)
- U2 pad 99: Net-(D4-Pad1) -> Net-(D3-Pad1)
Routing:
- net Net-(B55-Pad1): track 0.00 -> 15.4 mm, vias 0 -> 2
- net GND: track 115.1 -> 128.4 mm, vias 46 -> 51
- net Net-(J4-Pad1): track 0.00 -> 9.51 mm, vias 0 -> 1
- net Net-(B113-Pad1): track 0.00 -> 8.69 mm, vias 0 -> 3
- net Net-(J4-Pad2): track 0.00 -> 6.20 mm
- net Net-(B59-Pad1): track 0.00 -> 6.19 mm, vias 0 -> 1
- net Net-(R35-Pad2): track 0.00 -> 5.92 mm
- net Net-(B114-Pad1): track 0.00 -> 5.50 mm, vias 0 -> 1
- net Net-(B60-Pad1): track 0.00 -> 4.83 mm, vias 0 -> 1
- net Net-(R39-Pad1): track 0.00 -> 4.43 mm
- net Net-(B57-Pad1): track 0.00 -> 4.34 mm
- net Net-(B61-Pad1): track 0.00 -> 4.02 mm, vias 0 -> 1
- net Net-(B115-Pad1): track 0.00 -> 2.97 mm
- net Net-(R41-Pad2): track 0.00 -> 2.95 mm
- net Net-(R42-Pad2): track 0.00 -> 2.70 mm
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Other:
- board text added: "0cm"
- board text added: "10cm"
- board text added: "15cm"
- board text added: "2 LVDS pairs/IO"
- board text added: "4 IO or Jumpers"
- board text added: "4 LEDs"
- board text added: "5cm"
- board text added: "8cm"
- board text added: "AD9866"
- board text added: "Ethernet"
- board text added: "Ext PA Switch"
- board text added: "Ext Ref Clock"
- board text added: "Filters"
- board text added: "Instrument RX SMA"
- board text added: "Instrument TX SMA"
- board text added: "Main RX/TX"
- board text added: "OPA2677"
- board text added: "Power"
- board text added: "Power Supply"
- board text added: "Sync Rcvr Clock"
- board text added: "TX PA"

Commit message: More layout
Parts:
- added B116: 0.1uF, HERMESLITE:SMD-0603, F.Cu at (165.8, 84.2)
- added B72: 0.1uF, HERMESLITE:SMD-0603, B.Cu at (140.9, 171.8)
- added B73: 0.1uF, HERMESLITE:SMD-0603, F.Cu at (140.0, 171.3)
- added B74: 0.1uF, HERMESLITE:SMD-0603, B.Cu at (139.3, 170.2)
- added B86: 0.1uF, HERMESLITE:SMD-0603, B.Cu at (143.3, 170.3)
- added B87: 0.1uF, HERMESLITE:SMD-0603, B.Cu at (145.4, 170.3)
- added B88: 0.1uF, HERMESLITE:SMD-0603, B.Cu at (147.3, 170.3)
- added B89: 0.1uF, HERMESLITE:SMD-0603, B.Cu at (149.6, 166.0)
- added B90: 0.1uF, HERMESLITE:SMD-0603, B.Cu at (141.7, 161.7)
- added B91: 0.1uF, HERMESLITE:SMD-0603, B.Cu at (149.8, 163.6)
- added B92: 0.1uF, HERMESLITE:SMD-0603, B.Cu at (149.8, 161.5)
- added C13: 4.7nF, HERMESLITE:SMD-0603, B.Cu at (148.6, 72.3)
- added C14: 22uF, HERMESLITE:SMD-0805, B.Cu at (143.6, 66.8)
- added C15: 22uF, HERMESLITE:SMD-0805, B.Cu at (145.5, 66.8)
- added C16: 100uF, HERMESLITE:SMD-1210, F.Cu at (144.6, 67.0)
- added C17: 10uF, HERMESLITE:SMD-0805, F.Cu at (151.6, 63.0)
- added C18: 4.7uF, HERMESLITE:SMD-0805, F.Cu at (147.1, 72.7)
- added C19: 4.7nF, HERMESLITE:SMD-0603, B.Cu at (169.6, 72.5)
- added C20: 22uF, HERMESLITE:SMD-0805, B.Cu at (166.9, 67.2)
- added C21: 22uF, HERMESLITE:SMD-0805, B.Cu at (164.9, 67.2)
- added C22: 100uF, HERMESLITE:SMD-1210, F.Cu at (165.6, 67.2)
- added C23: 10uF, HERMESLITE:SMD-0805, F.Cu at (172.6, 63.1)
- added C24: 4.7uF, HERMESLITE:SMD-0805, F.Cu at (168.1, 72.8)
- added C25: 10uF, HERMESLITE:SMD-0603, F.Cu at (163.2, 83.4)
- added C26: 1uF, HERMESLITE:SMD-0603, F.Cu at (163.2, 89.3)
- added C48: 10uF, HERMESLITE:SMD-0805, F.Cu at (138.8, 172.5)
- added C60: 1uF, HERMESLITE:SMD-0603, B.Cu at (143.3, 173.0)
- added C61: 1uF, HERMESLITE:SMD-0603, B.Cu at (145.4, 173.0)
- added C62: 10uF, HERMESLITE:SMD-0603, B.Cu at (147.3, 173.2)
- added C63: 1uF, HERMESLITE:SMD-0603, B.Cu at (148.9, 170.3)
- added C64: 10uF, HERMESLITE:SMD-0603, B.Cu at (150.5, 170.3)
- added C65: 1uF, HERMESLITE:SMD-0603, B.Cu at (149.6, 167.6)
- added C66: 10uF, HERMESLITE:SMD-0603, B.Cu at (152.3, 166.0)
- added C67: 1uF, HERMESLITE:SMD-0603, B.Cu at (143.3, 161.7)
- added C68: 1uF, HERMESLITE:SMD-0603, B.Cu at (152.5, 163.6)
- added C69: 1uF, HERMESLITE:SMD-0603, B.Cu at (149.8, 159.9)
- added C70: 10uF, HERMESLITE:SMD-0603, B.Cu at (153.4, 161.6)
- added CL2: SMA, HERMESLITE:SMAVERT, F.Cu at (105.4, 128.7)
- added FB17: FB, HERMESLITE:SMD-0603, B.Cu at (149.6, 172.7)
- added FB18: FB, HERMESLITE:SMD-0603, B.Cu at (152.8, 170.3)
- added FB19: FB, HERMESLITE:SMD-0603, B.Cu at (152.3, 167.6)
- added FB20: FB, HERMESLITE:SMD-0603, B.Cu at (153.4, 159.9)
- added FB27: FB, HERMESLITE:SMD-0603, F.Cu at (149.2, 78.5)
- added FB28: DNI, HERMESLITE:SMD-0603, F.Cu at (149.2, 80.0)
- added FB29: DNI, HERMESLITE:SMD-0603, F.Cu at (149.2, 82.5)
- added FB30: FB, HERMESLITE:SMD-0603, F.Cu at (149.2, 84.0)
- added J11: JNC, HERMESLITE:SMD-0603, F.Cu at (174.5, 68.0)
- added J2: JNC, HERMESLITE:SMD-0603, F.Cu at (153.3, 68.0)
- added L1: 3.3uH, HERMESLITE:GENERICPSL, F.Cu at (146.3, 60.8)
- added L2: 2.2uH, HERMESLITE:GENERICPSL, F.Cu at (167.3, 60.9)
- added R11: 35.7K, HERMESLITE:SMD-0603, B.Cu at (148.6, 70.7)
- added R12: 11.5K, HERMESLITE:SMD-0603, B.Cu at (151.4, 70.7)
- added R13: DNI, HERMESLITE:SMD-0603, F.Cu at (153.9, 65.2)
- added R14: 20K, HERMESLITE:SMD-0603, B.Cu at (169.6, 70.8)
- added R15: 10K, HERMESLITE:SMD-0603, B.Cu at (172.4, 70.8)
- added R16: DNI, HERMESLITE:SMD-0603, F.Cu at (175.0, 65.3)
- added U16: ST1S10, HERMESLITE:ST1S10, F.Cu at (170.8, 68.0)
- added U17: TPS730, HERMESLITE:SOT23, F.Cu at (162.4, 87.7)
- added U3: ST1S10, HERMESLITE:ST1S10, F.Cu at (149.8, 68.0)
- added U7: AD9866BCPZ, HERMESLITE:AD9866, F.Cu at (145.3, 166.0)
- moved B58 56.4 mm to (123.5, 127.0)
- moved R44 50.7 mm to (120.7, 127.0)
- moved R43 50.6 mm to (117.9, 127.0)
- moved DB1 43.2 mm to (120.5, 130.3)
Connections:
- DB1 pad 1: Vclk -> +3V3
Routing:
- net Net-(L1-Pad1): track 0.00 -> 4.93 mm
- net +3V3: track 33.8 -> 38.4 mm
- net GND: track 128.4 -> 132.7 mm, vias 51 -> 53
- net Net-(J2-Pad2): track 0.00 -> 3.46 mm
- net Net-(C17-Pad1): track 0.00 -> 2.34 mm

Commit message: Additional layout work
Parts:
- added B83: 0.1uF, HERMESLITE:SMD-0603, F.Cu at (111.9, 121.3)
- added B84: 0.1uF, HERMESLITE:SMD-0603, F.Cu at (110.3, 121.3)
- added B85: 0.1uF, HERMESLITE:SMD-0603, F.Cu at (115.1, 121.3)
- added C58: 15pF, HERMESLITE:SMD-0603, F.Cu at (123.2, 109.7)
- added C59: 15pF, HERMESLITE:SMD-0603, F.Cu at (125.5, 112.8)
- added CL4: SMA, HERMESLITE:SMAVERT, F.Cu at (122.4, 102.2)
- added J10: JNC, HERMESLITE:SMD-0603, F.Cu at (119.9, 109.3)
- added J12: JNO, HERMESLITE:SMD-0603, B.Cu at (115.3, 128.2)
- added J16: JNO, HERMESLITE:SMD-0603, B.Cu at (107.1, 128.1)
- added J22: JNC, HERMESLITE:SMD-0603, B.Cu at (117.8, 102.2)
- added J7: JNO, HERMESLITE:SMD-0603, F.Cu at (119.8, 118.6)
- added J8: JNO, HERMESLITE:SMD-0603, F.Cu at (119.8, 120.8)
- added J9: JNC, HERMESLITE:SMD-0603, B.Cu at (121.5, 116.3)
- added R69: 1.6K, HERMESLITE:SMD-0603, F.Cu at (113.5, 121.3)
- added R70: 10K, HERMESLITE:SMD-0603, B.Cu at (120.7, 117.9)
- added T2: 8:1 Z, HERMESLITE:TRANSFSMT, F.Cu at (111.2, 127.2)
- added TP5: TEST_1P, HERMESLITE:TP, B.Cu at (106.6, 110.3)
- added TP6: TEST_1P, HERMESLITE:TP, F.Cu at (120.0, 111.4)
- added X3: 38.4MHz, HERMESLITE:XTAL, F.Cu at (123.0, 112.5)
- R43, R44: moved to B.Cu
- moved B89 61.9 mm to (117.4, 113.1)
- moved C65 61.9 mm to (117.4, 114.7)
- moved C70 61.9 mm to (120.4, 109.2)
- moved FB20 61.8 mm to (120.4, 107.6)
- moved C66 61.8 mm to (120.4, 113.1)
- moved FB19 61.8 mm to (120.4, 114.7)
- moved C68 61.7 mm to (120.4, 110.9)
- moved B72 61.6 mm to (108.4, 119.5)
- moved B86 61.5 mm to (111.1, 117.9)
- moved B88 61.5 mm to (115.1, 117.9)
- moved C48 61.5 mm to (106.6, 120.1)
- moved U7 61.5 mm to (113.1, 113.6)
- moved B73 61.5 mm to (107.8, 118.9)
- moved B87 61.5 mm to (113.2, 117.9)
- moved C63 61.5 mm to (116.7, 117.9)
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Connections:
- U2 pad 103: (no net) -> SDA
- U2 pad 104: (no net) -> SCL
- U7 pad 57: RFFE_CLK -> Net-(C58-Pad1)
Routing:
- net GND: track 132.7 -> 193.7 mm, vias 53 -> 56
- net Net-(U2-Pad105): track 0.00 -> 33.3 mm
- net Net-(U2-Pad106): track 0.00 -> 31.6 mm
- net RFFE_CLK: track 0.00 -> 29.8 mm, vias 0 -> 1
- net SDA: track 0.00 -> 27.7 mm
- net SCL: track 0.00 -> 27.0 mm
- net Net-(B90-Pad1): track 0.00 -> 25.7 mm, vias 0 -> 3
- net Net-(U2-Pad110): track 0.00 -> 24.7 mm
- net Net-(U2-Pad111): track 0.00 -> 23.9 mm
- net Net-(U2-Pad112): track 0.00 -> 23.1 mm
- net Net-(U2-Pad113): track 0.00 -> 22.2 mm
- net Net-(U2-Pad114): track 0.00 -> 21.4 mm
- net Net-(U2-Pad115): track 0.00 -> 20.6 mm
- net Net-(U2-Pad119): track 0.00 -> 19.1 mm
- net Net-(U2-Pad120): track 0.00 -> 17.6 mm
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Other:
- board text removed: "AD9866"
