File: hardware/hl/hermeslite.kicad_pcb (KiCad board)
At the start: 4 copper layers, 150 x 100 mm, 327 parts, among them CN1 USBBlaster2, CN3 MagJack, CN4 IO8, CN5 IO8, CN6 IO8, J1 JNC, J10 JNC, J11 JNC, J12 JNO, J13 JNO, J14 JNC, J15 JNC, J16 JNO, J17 JNO, J18 JNC, J2 JNC, J21 JNC, J22 JNC, J23 JNO, J3 JNO, J4 JNO, J5 JNO, J7 JNO, J8 JNO, J9 JNC, T2 8:1 Z, U1 EEPROM, U16 ST1S10, U17 TPS730, U2 FPGA, U3 ST1S10, U4 KSZ9031RN, U5 MCP4716, U6 5P49V5923, U7 AD9866BCPZ, X1 25MHz, X2 38.4MHz, X3 38.4MHz

Commit message: Latest filter values
Parts:
- removed the REF** at (139.8, 171.4)
- removed the REF** at (105.2, 165.5)
- removed the REF** at (90.0, 165.6)
- removed the REF** at (97.5, 163.8)
- removed the REF** at (152.3, 169.5)
- removed the REF** at (91.9, 157.9)
- removed the REF** at (126.0, 180.3)
- removed the REF** at (74.8, 165.5)
- removed the REF** at (137.3, 180.2)
- removed the REF** at (33.3, 173.9)
- removed the REF** at (46.5, 175.5)
- removed the REF** at (43.7, 163.5)
- removed the REF** at (38.8, 159.5)
- removed the REF** at (82.3, 163.8)
- removed the REF** at (125.8, 196.1)
- removed the REF** at (123.5, 188.3)
- removed the REF** at (111.5, 160.3)
- removed the REF** at (103.8, 157.8)
- added B68: 0.1uF, HERMESLITE:SMD-0603, F.Cu at (142.2, 115.6)
- added B75: 0.1uF, HERMESLITE:SMD-0603, B.Cu at (145.4, 120.9)
- added B78: 0.1uF, HERMESLITE:SMD-0603, F.Cu at (142.2, 120.8)
- added C49: 75pF, HERMESLITE:SMD-0805, F.Cu at (129.6, 118.2)
- added C50: 150pF, HERMESLITE:SMD-0805, F.Cu at (133.4, 118.2)
- added C51: 160pF, HERMESLITE:SMD-0805, F.Cu at (137.5, 118.2)
- added C52: 100pF, HERMESLITE:SMD-0805, F.Cu at (141.3, 118.2)
- added CN2: PS, HERMESLITE:POWER, F.Cu at (194.1, 152.7)
- added DB2: RFD4, HERMESLITE:4x1, F.Cu at (154.9, 114.3)
- added F1: 3A@20V, HERMESLITE:FUSE, F.Cu at (180.8, 157.2)
- added L4: 240nH, HERMESLITE:SMD-0805, F.Cu at (132.2, 115.5)
- added L5: 270nH, HERMESLITE:SMD-0805, F.Cu at (135.4, 115.2)
- added L6: 270nH, HERMESLITE:SMD-0805, F.Cu at (138.6, 115.5)
- added L7: 240nH, HERMESLITE:SMD-0805, F.Cu at (132.2, 120.9)
- added L8: 270nH, HERMESLITE:SMD-0805, F.Cu at (135.4, 121.2)
- added L9: 270nH, HERMESLITE:SMD-0805, F.Cu at (138.6, 120.9)
- added Q1: DMP3099L, HERMESLITE:SOT23_3, F.Cu at (169.1, 160.3)
- added R49: 2.2K, HERMESLITE:SMD-0603, B.Cu at (142.8, 111.3)
- added R50: 33, HERMESLITE:SMD-0603, F.Cu at (129.6, 115.1)
- added R51: 22, HERMESLITE:SMD-0603, F.Cu at (144.6, 114.8)
- added R55: 75, HERMESLITE:SMD-0603, B.Cu at (145.4, 116.5)
- added R56: 330, HERMESLITE:SMD-0603, F.Cu at (149.8, 113.0)
- added R57: 1K, HERMESLITE:SMD-0603, F.Cu at (135.3, 118.2)
- added R58: 1K, HERMESLITE:SMD-0603, F.Cu at (139.4, 118.2)
- added R59: 330, HERMESLITE:SMD-0603, F.Cu at (148.5, 123.2)
- added R63: 22, HERMESLITE:SMD-0603, F.Cu at (144.6, 121.5)
- added R64: 33, HERMESLITE:SMD-0603, F.Cu at (129.6, 121.3)
- added R65: 2.2K, HERMESLITE:SMD-0603, B.Cu at (140.7, 111.4)
- added REF**: inductor, HERMESLITE:inductorrev, F.Cu at (129.4, 155.4)
- added REF**: inductor, HERMESLITE:inductor, F.Cu at (99.5, 203.9)
- added REF**: inductor, HERMESLITE:inductor, F.Cu at (80.9, 202.7)
- added REF**: inductor, HERMESLITE:inductor, F.Cu at (69.4, 200.7)
- added REF**: inductor, HERMESLITE:inductorrev, F.Cu at (78.2, 155.5)
- added REF**: inductor, HERMESLITE:inductor, F.Cu at (75.3, 164.6)
- added REF**: inductor, HERMESLITE:inductor, F.Cu at (90.5, 164.6)
- added REF**: inductor, HERMESLITE:inductorrev, F.Cu at (91.6, 155.5)
- added REF**: inductor, HERMESLITE:inductor, F.Cu at (114.8, 160.6)
- added REF**: inductor, HERMESLITE:inductor, F.Cu at (105.7, 164.6)
- added REF**: inductor, HERMESLITE:inductorrev, F.Cu at (104.6, 155.5)
- added REF**: Val**, HERMESLITE:SMD-0805, F.Cu at (39.7, 176.9)
- added REF**: inductor, HERMESLITE:inductorrev, F.Cu at (66.1, 154.2)
- added REF**: inductor, HERMESLITE:inductor, F.Cu at (68.4, 163.3)
- added REF**: inductor, HERMESLITE:inductorrev, F.Cu at (111.8, 196.9)
- added REF**: inductor, HERMESLITE:inductorrev, F.Cu at (98.6, 196.9)
- added REF**: inductor, HERMESLITE:inductorrev, F.Cu at (84.5, 196.8)
- added REF**: inductor, HERMESLITE:inductorrev, F.Cu at (70.7, 196.8)
- added REF**: inductor, HERMESLITE:inductor, F.Cu at (125.7, 187.1)
- added U9: OPA2677, HERMESLITE:OPA2677, F.Cu at (150.4, 115.2)
- moved REF** 74.6 mm to (60.8, 185.9), turned to 90 degrees
- moved REF** 59.1 mm to (68.4, 175.6), turned to 270 degrees
- moved REF** 2.60 mm to (114.0, 175.6)
- moved REF** 0.10 mm to (98.8, 175.6)
- moved REF** 0.10 mm to (83.6, 175.6)

Commit message: Updated schematics
Parts:
- removed CL4: SMA, HERMESLITE:SMAVERT
- removed DB6: RFD4b, HERMESLITE:4x1
- removed REF** (x9): inductor, HERMESLITE:inductorrev
- removed REF** (x9): inductor, HERMESLITE:inductor
- removed REF** (x8): DPDT, HERMESLITE:DPDT
- removed REF**: Val**, HERMESLITE:SMD-0805
- removed RF4: BNC, HERMESLITE:SMAVERT
- added B100: 0.1uF, HERMESLITE:SMD-0603, F.Cu at (208.3, 114.0)
- added B101: 0.1uF, HERMESLITE:SMD-0603, F.Cu at (212.7, 114.2)
- added B102: 0.1uF, HERMESLITE:SMD-0603, F.Cu at (216.5, 114.6)
- added B103: 0.1uF, HERMESLITE:SMD-0603, F.Cu at (211.7, 118.0)
- added B104: 0.1uF, HERMESLITE:SMD-0603, B.Cu at (158.2, 129.7)
- added B105: 0.1uF, HERMESLITE:SMD-0603, F.Cu at (138.4, 129.2)
- added B106: 0.1uF, HERMESLITE:SMD-0603, B.Cu at (146.8, 129.1)
- added B107: 0.1uF, HERMESLITE:SMD-0603, B.Cu at (141.2, 129.7)
- added B108: 0.1uF, HERMESLITE:SMD-0603, F.Cu at (145.0, 150.1)
- added B97: 0.1uF, HERMESLITE:SMD-0603, F.Cu at (155.4, 129.2)
- added B98: 0.1uF, HERMESLITE:SMD-0603, F.Cu at (153.8, 120.0)
- added B99: 0.1uF, HERMESLITE:SMD-0603, B.Cu at (160.2, 127.4)
- added C148: DNI, HERMESLITE:SMD-0805, B.Cu at (155.7, 130.2)
- added C149: DNI, HERMESLITE:SMD-0805, B.Cu at (138.7, 130.2)
- added D6: DNI, HERMESLITE:SOT23_3, B.Cu at (151.4, 130.5)
- added D7: DNI, HERMESLITE:SOT23_3, B.Cu at (134.4, 130.5)
- added L33: 100nH, HERMESLITE:SMD-0805, F.Cu at (161.0, 129.9)
- added L34: 100nH, HERMESLITE:SMD-0805, F.Cu at (144.0, 129.9)
- added MH: VAL**, HERMESLITE:m1p6, F.Cu at (148.3, 133.3)
- added Q3: LDMOS, HERMESLITE:COMBORF, F.Cu at (156.8, 140.0)
- added Q4: LDMOS, HERMESLITE:COMBORF, F.Cu at (139.8, 140.0)
- added R100: 10, HERMESLITE:SMD-0805, B.Cu at (200.2, 149.9)
- added R101: 1K, HERMESLITE:SMD-0805, B.Cu at (143.7, 129.2)
- added R92: 270, HERMESLITE:SMD-0805, F.Cu at (158.4, 129.2)
- added R93: DNI, HERMESLITE:SMD-0805, F.Cu at (209.3, 119.7)
- added R94: 10, HERMESLITE:SMD-0805, B.Cu at (200.2, 147.6)
- added R95: 1K, HERMESLITE:SMD-0805, B.Cu at (160.7, 129.2)
- added R96: DNI, HERMESLITE:SMD-0805, F.Cu at (214.2, 120.6)
- added R97: DNI, HERMESLITE:SMD-0805, B.Cu at (197.4, 148.8)
- added R98: DNI, HERMESLITE:SMD-0805, B.Cu at (202.9, 148.8)
- added R99: 270, HERMESLITE:SMD-0805, F.Cu at (141.4, 129.2)
- added T3: TRANSF4CTS, HERMESLITE:BN202V, F.Cu at (145.5, 123.3)
- moved CN2 134.1 mm to (247.8, 29.8), turned to 180 degrees
- moved R65 11.5 mm to (144.8, 100.7)
- moved R49 11.5 mm to (146.9, 100.5)
- moved B75 8.22 mm to (147.1, 112.8)
- moved L7 8.22 mm to (133.8, 112.8)
- moved L9 8.22 mm to (140.2, 112.8)
- moved B68 8.22 mm to (143.8, 107.5)
- moved B78 8.22 mm to (143.8, 112.8)
- moved C49 8.22 mm to (131.2, 110.2)
- moved C50 8.22 mm to (135.1, 110.2)
- moved C51 8.22 mm to (139.2, 110.2)
- moved DB2 8.22 mm to (156.6, 106.2)
- moved L4 8.22 mm to (133.8, 107.5)
- moved L5 8.22 mm to (137.1, 107.2)
- moved L6 8.22 mm to (140.2, 107.5)
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Routing:
- net Net-(B97-Pad1): track 0.00 -> 11.9 mm
- net Net-(B105-Pad1): track 0.00 -> 11.9 mm
- net Net-(B99-Pad2): track 0.00 -> 9.91 mm
- net Net-(B106-Pad2): track 0.00 -> 8.56 mm
- net Net-(B106-Pad1): track 0.00 -> 2.89 mm, vias 0 -> 1
- net Net-(B99-Pad1): track 0.00 -> 2.77 mm, vias 0 -> 1
Other:
- board text removed: "Add power supply taps 3.3, 2.5, 1.2"
- board text removed: "Filters"
- board text removed: "OPA2677"
- board text removed: "TX PA"

Commit message: More layout
Parts:
- added B109: 0.1uF, HERMESLITE:SMD-0603, F.Cu at (130.8, 126.2)
- added B110: 0.1uF, HERMESLITE:SMD-0603, F.Cu at (147.6, 124.5)
- added B111: 0.1uF, HERMESLITE:SMD-0603, F.Cu at (140.5, 98.8)
- added B66: 0.1uF, HERMESLITE:SMD-0603, B.Cu at (152.1, 102.8)
- added B69: 0.1uF, HERMESLITE:SMD-0603, F.Cu at (155.0, 108.1)
- added B70: 0.1uF, HERMESLITE:SMD-0603, F.Cu at (149.8, 105.5)
- added B71: 0.1uF, HERMESLITE:SMD-0603, B.Cu at (154.3, 103.8)
- added B76: 0.1uF, HERMESLITE:SMD-0603, F.Cu at (154.3, 116.1)
- added B77: 0.1uF, HERMESLITE:SMD-0603, F.Cu at (149.8, 113.5)
- added B79: 0.1uF, HERMESLITE:SMD-0603, B.Cu at (154.0, 111.5)
- added B80: 0.1uF, HERMESLITE:SMD-0603, B.Cu at (138.7, 106.6)
- added B81: 0.1uF, HERMESLITE:SMD-0603, B.Cu at (126.0, 124.1)
- added B82: 0.1uF, HERMESLITE:SMD-0603, B.Cu at (163.1, 117.2)
- added C144: 1uF, HERMESLITE:SMD-0805, B.Cu at (132.7, 103.8)
- added C145: 1uF, HERMESLITE:SMD-0805, B.Cu at (132.7, 112.8)
- added C146: 1uF, HERMESLITE:SMD-0805, B.Cu at (132.7, 105.8)
- added C147: 1uF, HERMESLITE:SMD-0805, B.Cu at (132.7, 114.8)
- added C150: 10uF, HERMESLITE:SMD-0805, F.Cu at (138.0, 97.7)
- added C151: 1uF, HERMESLITE:SMD-0805, B.Cu at (132.7, 100.8)
- added C27: 4.7nF, HERMESLITE:SMD-0603, F.Cu at (145.9, 68.2)
- added C28: 22uF, HERMESLITE:SMD-0805, F.Cu at (144.9, 58.7)
- added C29: 22uF, HERMESLITE:SMD-0805, F.Cu at (144.9, 60.5)
- added C30: 22uF, HERMESLITE:SMD-0805, F.Cu at (144.9, 62.2)
- added C31: 22uF, HERMESLITE:SMD-0805, F.Cu at (141.6, 57.3)
- added C32: 22uF, HERMESLITE:SMD-0805, F.Cu at (141.6, 59.2)
- added C33: 10uF, HERMESLITE:SMD-1206, F.Cu at (150.1, 59.0)
- added C34: 4.7uF, HERMESLITE:SMD-0805, B.Cu at (152.0, 67.7)
- added C43: 10uF, HERMESLITE:SMD-1206, F.Cu at (149.2, 85.7)
- added C46: 1uF, HERMESLITE:SMD-0805, F.Cu at (160.8, 84.9)
- added C53: 10pF, HERMESLITE:SMD-0805, B.Cu at (118.3, 129.3)
- added C54: DNI, HERMESLITE:SMD-0805, B.Cu at (121.3, 128.6)
- added C55: 100pF, HERMESLITE:SMD-0805, B.Cu at (117.6, 126.7)
- added C56: 180pF, HERMESLITE:SMD-0805, B.Cu at (122.1, 131.5)
- added C57: 100pF, HERMESLITE:SMD-0805, B.Cu at (121.3, 125.3)
- added C81: 100pF, HERMESLITE:SMD-0805, F.Cu at (155.2, 121.8)
- added CL4: RFD2b, HERMESLITE:2x1, F.Cu at (118.7, 100.8)
- added CN11: RFD2b, HERMESLITE:2x1, F.Cu at (168.4, 97.0)
- added DB10: RFD2b, HERMESLITE:2x1, F.Cu at (154.4, 56.5)
- added DB11: RFD2b, HERMESLITE:2x1, F.Cu at (125.5, 68.8)
- added DB12: RFD2b, HERMESLITE:2x1, F.Cu at (113.9, 64.4)
- added DB13: RFD2b, HERMESLITE:2x1, F.Cu at (154.9, 68.8)
- added DB14: RFD2b, HERMESLITE:2x1, F.Cu at (143.3, 64.4)
- added DB15: RFD2b, HERMESLITE:2x1, F.Cu at (151.2, 72.4)
- added DB16: RFD2a, HERMESLITE:2x1, F.Cu at (115.2, 130.1)
- added DB18: RFD2b, HERMESLITE:2x1, F.Cu at (154.3, 165.2)
- added DB19: RFD4b, HERMESLITE:4x1, F.Cu at (144.9, 155.7)
- added DB20: RFD2b, HERMESLITE:2x1, F.Cu at (152.9, 108.9)
- added DB21: RFD2b, HERMESLITE:2x1, F.Cu at (159.1, 104.8)
- added DB23: RFD2b, HERMESLITE:2x1, F.Cu at (152.1, 116.6)
- added DB25: RFD2b, HERMESLITE:2x1, F.Cu at (157.3, 115.5)
- added DB26: RFD2b, HERMESLITE:2x1, F.Cu at (160.1, 63.4)
- added DB27: RFD2b, HERMESLITE:2x1, F.Cu at (127.5, 52.0)
- added DB4: RFD2a, HERMESLITE:2x1, F.Cu at (123.7, 125.5)
- added DB6: RFD2b, HERMESLITE:2x1, F.Cu at (117.6, 119.2)
- added DB8: RFD2b, HERMESLITE:2x1, F.Cu at (140.2, 68.8)
- added DB9: RFD2b, HERMESLITE:2x1, F.Cu at (128.6, 64.4)
- added FB14: FB, HERMESLITE:SMD-0603, B.Cu at (150.4, 102.8)
- added FB15: FB, HERMESLITE:SMD-0603, F.Cu at (147.6, 71.0)
- added J19: JNC, HERMESLITE:SMD-0603, F.Cu at (154.2, 63.5)
- added J20: JNC, HERMESLITE:SMD-0603, F.Cu at (152.9, 82.3)
- added J6: DNI, HERMESLITE:2x1, F.Cu at (142.9, 54.5)
- added K2: NA3WK-K, HERMESLITE:DPDT_GND, F.Cu at (160.1, 124.4)
- added L10: 330nH, HERMESLITE:SMD-0805, B.Cu at (118.3, 131.5)
- added L11: 330nH, HERMESLITE:SMD-0805, B.Cu at (123.6, 128.6)
- added L3: 3.3uH, HERMESLITE:GENERICPSL, F.Cu at (148.1, 54.6)
- added Q2: NUD3124, HERMESLITE:SOT23_3, B.Cu at (163.6, 98.3)
- added Q5: 2N7002K, HERMESLITE:SOT23_3, F.Cu at (165.2, 98.3)
- added R102: 1.6K, HERMESLITE:SMD-0603, F.Cu at (150.5, 89.0)
- added R123: 4.7K, HERMESLITE:SMD-0603, F.Cu at (161.5, 160.1)
- added R124: 4.7K, HERMESLITE:SMD-0603, F.Cu at (159.8, 163.1)
- added R125: DNI, HERMESLITE:SMD-0603, F.Cu at (165.5, 100.0)
- added R19: 16.2K, HERMESLITE:SMD-0603, F.Cu at (145.9, 66.6)
- added R46: 1.5K, HERMESLITE:SMD-0603, F.Cu at (151.8, 68.2)
- added R47: DNI, HERMESLITE:SMD-0603, F.Cu at (154.7, 61.1)
- added R52: 10, HERMESLITE:SMD-0805, F.Cu at (147.2, 103.4)
- added R54: 14, HERMESLITE:SMD-0805, B.Cu at (156.6, 104.6)
- added R61: 14, HERMESLITE:SMD-0805, B.Cu at (156.4, 110.7)
- added R62: 10, HERMESLITE:SMD-0805, F.Cu at (146.2, 115.6)
- added R67: 1K, HERMESLITE:SMD-0603, B.Cu at (140.1, 102.5)
- added R68: 1K, HERMESLITE:SMD-0603, B.Cu at (137.4, 102.5)
- added R91: 12.1K, HERMESLITE:SMD-0603, F.Cu at (151.3, 86.0)
- added RF1: BNC, HERMESLITE:SMAEDGE_TH, F.Cu at (169.9, 106.2)
- added RF2: BNC, HERMESLITE:SMAEDGE_TH, F.Cu at (169.9, 128.2)
- added RF3: BNC, HERMESLITE:SMAEDGE_TH, B.Cu at (169.9, 117.2)
- added T1: 1:1 Z, HERMESLITE:TRANSFSMT4, F.Cu at (160.0, 110.2)
- added U10: PE4259, HERMESLITE:PE4259, F.Cu at (153.9, 106.2)
- added U11: PE4259, HERMESLITE:PE4259, F.Cu at (153.9, 114.2)
- added U12: AP2204, HERMESLITE:ap2204, F.Cu at (155.9, 85.8)
- added U14: LP2985, HERMESLITE:SOT23, F.Cu at (137.0, 102.2)
- added U15: MCP4661, HERMESLITE:MCP4661, F.Cu at (130.0, 101.1)
- added U8: ST1S10, HERMESLITE:ST1S10, F.Cu at (150.7, 63.8)
- B106, B99, R100, R94, R97, R98: moved to F.Cu
- B108, B98, C15, R93, R96: moved to B.Cu
- CN2: footprint HERMESLITE:POWER -> HERMESLITE:POWERPP
- DB2: value RFD4 -> RFD4d
- DB3: value RFD4b -> RFD4d
- MH (x4): footprint HERMESLITE:MH -> HERMESLITE:m2p5
- MH: footprint HERMESLITE:m1p6 -> HERMESLITE:m2p0
- moved Q1 107.9 mm to (155.6, 53.2), turned to 270 degrees
- moved F1 104.2 mm to (163.6, 54.4), turned to 180 degrees
- moved CN2 91.8 mm to (162.4, 63.4)
- moved R96 81.2 mm to (133.1, 124.0), turned to 90 degrees
- moved B102 79.5 mm to (137.1, 118.4)
- moved B100 73.0 mm to (135.3, 116.7)
- moved B101 72.9 mm to (139.8, 116.7), turned to 180 degrees
- moved B103 71.2 mm to (140.5, 118.4), turned to 180 degrees
- moved R93 64.5 mm to (144.9, 124.0), turned to 270 degrees
- moved R100 56.9 mm to (149.4, 124.5), turned to 90 degrees
- moved R98 56.6 mm to (150.6, 127.2), turned to 0 degrees
- moved R97 54.0 mm to (150.6, 121.8), turned to 0 degrees
- moved R94 53.7 mm to (151.8, 124.5), turned to 90 degrees
- moved B108 52.3 mm to (130.2, 99.9), turned to 270 degrees
- moved MH 50.0 mm to (167.0, 48.3)
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Connections:
- net +IOV renamed +VPA
- net SCL renamed /Clock/SCL1
- net SDA renamed /Clock/SDA1
- B98 pad 1: TXFILTER -> Net-(B98-Pad1)
- DB2 pad 1: /RF Frontend/Vop -> Net-(B70-Pad2)
- DB2 pad 2: Net-(DB2-Pad2) -> GND
- DB2 pad 3: Net-(DB2-Pad3) -> GND
- DB2 pad 4: GND -> Net-(B77-Pad2)
- DB3 pad 2: Net-(C49-Pad1) -> GND
- DB3 pad 4: GND -> Net-(C49-Pad1)
- R13 pad 2: Net-(DB23-Pad3) -> Net-(DB8-Pad1)
- R16 pad 2: Net-(DB23-Pad2) -> Net-(DB11-Pad1)
- R56 pad 1: Net-(DB2-Pad2) -> Net-(R52-Pad2)
- R59 pad 1: Net-(DB2-Pad3) -> Net-(R59-Pad1)
- R64 pad 1: Net-(C49-Pad2) -> GND
- R64 pad 2: GND -> Net-(C49-Pad2)
- U2 pad 11: (no net) -> Net-(FB14-Pad2)
- U2 pad 39: (no net) -> Net-(U14-Pad3)
- U2 pad 42: (no net) -> Net-(FB15-Pad1)
- U2 pad 43: (no net) -> Net-(DB13-Pad1)
- U2 pad 44: (no net) -> Net-(DB8-Pad1)
- U2 pad 46: (no net) -> Net-(DB11-Pad1)
- U9 pad 1: Net-(DB2-Pad2) -> Net-(R52-Pad2)
- U9 pad 7: Net-(DB2-Pad3) -> Net-(R59-Pad1)
- U9 pad 8: /RF Frontend/Vop -> +VOP
Routing:
- net +VPA: track 0.00 -> 113.6 mm, vias 0 -> 5
- net GND: track 368.1 -> 473.1 mm, vias 144 -> 171
- net Net-(DB13-Pad1): track 0.00 -> 54.1 mm
- net +VOP: track 0.00 -> 52.7 mm, vias 0 -> 1
- net Net-(C17-Pad1): track 69.9 -> 118.7 mm, vias 4 -> 6
- net PATRRX: track 0.00 -> 47.4 mm
- net /PA/bias0: track 0.36 -> 46.3 mm, vias 0 -> 2
- net (no net): track 151.7 -> 106.8 mm
- net Net-(DB8-Pad1): track 0.00 -> 40.3 mm
- net Net-(U14-Pad3): track 0.00 -> 35.1 mm, vias 0 -> 1
- net /PA/bias1: track 0.00 -> 30.1 mm, vias 0 -> 2
- net Net-(DB11-Pad1): track 0.00 -> 26.2 mm
- net Net-(CN2-Pad1): track 0.00 -> 24.7 mm
- net Net-(C81-Pad1): track 0.00 -> 23.2 mm, vias 0 -> 1
- net Net-(B98-Pad1): track 0.00 -> 22.5 mm
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Other:
- board size 150 x 100 mm -> 100 x 100 mm
- board text added: "Extra IO Slow Analog Inputs"
- board text added: "Low Power TX"
- board text added: "Optional RX Only"
- board text added: "PTT Out"
- board text added: "RX/TX Switched"
- board text removed: "10V Power Supply"
- board text removed: "15cm"
- board text removed: "5cm"
- board text removed: "8cm"
- board text removed: "Ext PA Switch"
- board text removed: "Instrument RX SMA"
- board text removed: "Instrument TX SMA"
- board text removed: "Main RX/TX"
- board text removed: "Slow ADC? Digital Bias? Bus Expander?"

Commit message: Latest layout
Parts:
- removed R123, R124: 4.7K, HERMESLITE:SMD-0603
- added B117: 0.1uF, HERMESLITE:SMD-0603, F.Cu at (147.2, 85.8)
- added B67: 0.1uF, HERMESLITE:SMD-0603, F.Cu at (147.2, 77.8)
- added B93: 0.1uF, HERMESLITE:SMD-0603, B.Cu at (147.2, 79.4)
- added B94: 0.1uF, HERMESLITE:SMD-0603, B.Cu at (143.0, 85.0)
- added B95: 0.1uF, HERMESLITE:SMD-0603, B.Cu at (147.2, 84.2)
- added B96: 0.1uF, HERMESLITE:SMD-0603, B.Cu at (154.0, 81.9)
- added C47: 1uF, HERMESLITE:SMD-0603, F.Cu at (158.1, 97.9)
- added C79: 1uF, HERMESLITE:SMD-0603, F.Cu at (152.4, 97.9)
- added C80: 1uF, HERMESLITE:SMD-0603, F.Cu at (146.7, 97.9)
- added C82: DNI, HERMESLITE:SMD-0603, F.Cu at (160.9, 84.0)
- added C83: DNI, HERMESLITE:SMD-0603, F.Cu at (163.1, 88.1)
- added CN10: RFD2b, HERMESLITE:2x1, F.Cu at (149.5, 95.8)
- added CN12: RFD2b, HERMESLITE:2x1, F.Cu at (168.4, 70.6)
- added CN7: IO8, HERMESLITE:IO, F.Cu at (167.3, 82.2)
- added CN8: RFD2b, HERMESLITE:2x1, F.Cu at (160.9, 95.8)
- added CN9: RFD2b, HERMESLITE:2x1, F.Cu at (155.2, 95.8)
- added D10: 1N5711, HERMESLITE:1N5711WS, B.Cu at (156.7, 78.6)
- added D11: 1N5711, HERMESLITE:1N5711WS, B.Cu at (156.7, 85.0)
- added D8: 1N5711, HERMESLITE:1N5711WS, B.Cu at (151.3, 85.0)
- added D9: 1N5711, HERMESLITE:1N5711WS, B.Cu at (151.3, 78.6)
- added DB17: RFD4b, HERMESLITE:4x1, F.Cu at (140.9, 77.3)
- added DB28: RFD2b, HERMESLITE:2x1, F.Cu at (147.5, 75.6)
- added J24: JNC, HERMESLITE:SMD-0603, F.Cu at (163.1, 84.7)
- added J25: JNC, HERMESLITE:SMD-0603, F.Cu at (163.1, 86.4)
- added J26: JNC, HERMESLITE:SMD-0603, F.Cu at (163.0, 81.2)
- added J27: JNC, HERMESLITE:SMD-0603, F.Cu at (163.5, 78.4)
- added R103: 1K, HERMESLITE:SMD-0603, B.Cu at (150.2, 75.7)
- added R104: 1.8K, HERMESLITE:SMD-0603, B.Cu at (147.2, 77.8)
- added R105: 220K, HERMESLITE:SMD-0603, B.Cu at (153.2, 84.2)
- added R106: 4.7K, HERMESLITE:SMD-0603, B.Cu at (143.0, 79.1)
- added R107: 4.7K, HERMESLITE:SMD-0603, B.Cu at (143.0, 82.0)
- added R108: 1K, HERMESLITE:SMD-0603, B.Cu at (149.3, 79.3)
- added R109: 1.8K, HERMESLITE:SMD-0603, B.Cu at (147.2, 81.0)
- added R110: 220K, HERMESLITE:SMD-0603, B.Cu at (153.2, 79.4)
- added R111: 1K, HERMESLITE:SMD-0603, B.Cu at (149.3, 84.3)
- added R112: 1.8K, HERMESLITE:SMD-0603, B.Cu at (147.2, 82.6)
- added R113: 220K, HERMESLITE:SMD-0603, B.Cu at (154.8, 79.4)
- added R114: 1K, HERMESLITE:SMD-0603, B.Cu at (150.2, 87.9)
- added R115: 1.8K, HERMESLITE:SMD-0603, B.Cu at (147.2, 85.8)
- added R116: 220K, HERMESLITE:SMD-0603, B.Cu at (154.8, 84.2)
- added R117: 10K, HERMESLITE:SMD-0603, B.Cu at (157.6, 98.4)
- added R118: 10K, HERMESLITE:SMD-0603, B.Cu at (151.9, 98.4)
- added R119: 10K, HERMESLITE:SMD-0603, B.Cu at (146.2, 98.4)
- added R120: 330, HERMESLITE:SMD-0603, F.Cu at (158.1, 95.4)
- added R121: 330, HERMESLITE:SMD-0603, F.Cu at (152.4, 95.4)
- added R122: 330, HERMESLITE:SMD-0603, F.Cu at (146.7, 95.4)
- added R48: 4.7K, HERMESLITE:SMD-0603, B.Cu at (142.7, 93.7)
- added R53: 4.7K, HERMESLITE:SMD-0603, B.Cu at (143.9, 96.9)
- added U13: MAX11613, HERMESLITE:MAX11613, F.Cu at (145.5, 81.8)
- added U18: LMV324, HERMESLITE:LMV324, F.Cu at (154.0, 81.8)
- B66, FB14: moved to F.Cu
- C43, C46, J20: moved to B.Cu
- DB19: value RFD4b -> RFD2b; footprint HERMESLITE:4x1 -> HERMESLITE:2x1
- moved DB18 68.9 mm to (165.9, 97.3)
- moved DB19 67.8 mm to (147.5, 88.0), turned to 180 degrees
- moved DB15 66.4 mm to (215.8, 87.5), turned to 180 degrees
- moved J20 16.0 mm to (139.1, 74.2), turned to 270 degrees
- moved R102 15.0 mm to (155.7, 74.9)
- moved R91 14.1 mm to (156.2, 72.8)
- moved C46 13.8 mm to (166.1, 72.2)
- moved C43 13.7 mm to (156.7, 74.2), turned to 0 degrees
- moved U12 13.3 mm to (160.7, 73.4)
- moved CN11 5.60 mm to (168.4, 91.4)
- moved Q2 5.60 mm to (163.6, 92.7)
- moved Q5 5.60 mm to (165.2, 92.7)
- moved R125 5.60 mm to (165.5, 94.4)
- moved B108 2.05 mm to (131.7, 98.5)
- moved C151 0.60 mm to (132.7, 101.4)
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Connections:
- DB19 pad 1: +3V3 -> Net-(DB19-Pad1)
- DB19 pad 2: /PA/SDA2 -> GND
- U15 pad 2: /PA/SCL2 -> SCL2
- U15 pad 3: /PA/SDA2 -> SDA2
- U2 pad 23: (no net) -> Net-(C80-Pad1)
- U2 pad 24: (no net) -> Net-(C79-Pad1)
- U2 pad 25: (no net) -> Net-(C47-Pad1)
- U2 pad 28: (no net) -> /PA/TR
- U2 pad 30: (no net) -> SDA2
- U2 pad 31: (no net) -> SCL2
- U2 pad 32: (no net) -> Net-(DB17-Pad3)
- U2 pad 33: (no net) -> Net-(DB17-Pad2)
Routing:
- net +3V3: track 430.6 -> 572.4 mm, vias 27 -> 38
- net (no net): track 106.8 -> 0.00 mm
- net GND: track 473.1 -> 558.5 mm, vias 171 -> 201
- net SDA2: track 0.00 -> 84.1 mm, vias 0 -> 2
- net SCL2: track 0.00 -> 82.0 mm, vias 0 -> 2
- net /PA/TR: track 0.00 -> 67.9 mm
- net Net-(C47-Pad1): track 0.00 -> 56.0 mm, vias 0 -> 1
- net Net-(C79-Pad1): track 0.00 -> 49.9 mm, vias 0 -> 1
- net Net-(C80-Pad1): track 0.00 -> 43.8 mm, vias 0 -> 1
- net +VPA: track 113.6 -> 157.1 mm, vias 5 -> 6
- net Net-(FB15-Pad1): track 0.00 -> 35.9 mm
- net Net-(DB17-Pad2): track 0.00 -> 30.4 mm
- net Net-(DB17-Pad3): track 0.00 -> 29.6 mm
- net Net-(FB14-Pad2): track 19.2 -> 43.7 mm, vias 0 -> 2
- net Net-(DB15-Pad1): track 1.53 -> 24.7 mm, vias 1 -> 2
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
Commit message: Before silk cleanup
Parts:
- removed DB15: RFD2b, HERMESLITE:2x1
- added TP1: TEST_1P, HERMESLITE:TP, F.Cu at (152.1, 71.7)
- moved FB10 0.20 mm to (109.4, 50.7)
- moved FB29 0.20 mm to (109.4, 52.3)
- moved C39 0.15 mm to (106.6, 51.1)
Routing:
- net GND: track 558.5 -> 567.8 mm
- net Net-(B42-Pad1): track 33.4 -> 30.8 mm
- net Net-(DB17-Pad3): track 29.6 -> 32.2 mm
- net Net-(FB15-Pad2): track 24.7 -> 25.5 mm
- net /PA/TR: track 67.9 -> 68.6 mm
- added copper zone on In2.Cu, net GND
Other:
- outline, holes or cut-outs redrawn
