File: hardware/hl/hermeslite.kicad_pcb (KiCad board)
At the start: 4 copper layers, 100 x 100 mm, 508 parts, among them CN1 USBBlaster2, CN10 RFD2b, CN11 RFD2b, CN12 RFD2b, CN2 PS, CN3 MagJack, CN4 IO8, CN5 IO8, CN6 IO8, CN7 IO8, CN8 RFD2b, CN9 RFD2b, J1 JNC, J10 JNC, J11 JNC, J12 JNO, J13 JNO, J14 JNC, J15 JNC, J16 JNO, J17 JNO, J18 JNC, J19 JNC, J2 JNC, J20 JNC, J21 JNC, J22 JNC, J23 JNO, J24 JNC, J25 JNC, J26 JNC, J27 JNC, J28 JNO, J3 JNO, J4 JNO, J5 JNO, J6 DNI, J7 JNO, J8 JNO, J9 JNC, K2 NA3WK-K, Q1 DMP3099L, Q2 NUD3124, Q3 LDMOS, Q4 LDMOS, Q5 2N7002K, T1 1:1 Z, T2 8:1 Z, T3 TRANSF4CTS, U1 EEPROM, U10 PE4259, U11 PE4259, U12 AP2204, U13 MAX11613, U14 LP2985, U15 MCP4661, U16 ST1S10, U17 TPS730, U18 LMV324, U2 FPGA, U3 ST1S10, U4 KSZ9031RN, U5 MCP4716, U6 5P49V5923, U7 AD9866BCPZ, U8 ST1S10, U9 OPA2677, X1 25MHz, X2 38.4MHz, X3 38.4MHz

Commit message: Before clock rework
Parts:
- removed DB7: RFD2b, HERMESLITE:2x1
- added B118: DNI, HERMESLITE:SMD-0603, B.Cu at (148.0, 90.4)
- added B119: 0.1uF, HERMESLITE:SMD-0603, B.Cu at (152.9, 106.4)
- added B120: 0.1uF, HERMESLITE:SMD-0603, B.Cu at (152.7, 114.4)
- added B121: DNI, HERMESLITE:SMD-0603, F.Cu at (122.8, 135.1)
- added J29: JNC, HERMESLITE:SMD-0603, B.Cu at (150.2, 89.6)
- added Q6: MCP9700, HERMESLITE:SOT23_3, F.Cu at (159.2, 135.0)
- added Q7: MCP9700, HERMESLITE:SOT23_3, F.Cu at (124.4, 135.0)
- added TP2: TEST_1P, HERMESLITE:TP, F.Cu at (106.4, 71.7)
- added TP3: TEST_1P, HERMESLITE:1x1, F.Cu at (115.2, 133.2)
- B71: moved to F.Cu
- DB21, DB25: value RFD2b -> TEST_1P; footprint HERMESLITE:2x1 -> HERMESLITE:1x1
- moved R125 3.89 mm to (162.7, 91.7), turned to 270 degrees
- moved Q2 1.65 mm to (165.2, 93.1), turned to 0 degrees
- moved B71 1.21 mm to (155.4, 103.3)
- moved D6 0.92 mm to (145.5, 131.2), turned to 180 degrees
- moved D7 0.92 mm to (128.5, 131.2), turned to 180 degrees
- moved DB21 0.50 mm to (158.5, 104.8), turned to 0 degrees
- moved B66 0.50 mm to (151.6, 102.8)
- moved FB14 0.50 mm to (149.9, 102.8)
- moved Q5 0.40 mm to (165.2, 93.1)
- moved R54 0.32 mm to (156.3, 104.7)
- moved DB25 0.30 mm to (157.2, 115.5)
- moved B100 0.20 mm to (135.1, 116.7)
Connections:
- D6 pad 1: GND -> Net-(B97-Pad1)
- D6 pad 2: Net-(B97-Pad1) -> GND
- D7 pad 1: GND -> Net-(B105-Pad1)
- D7 pad 2: Net-(B105-Pad1) -> GND
- Q1 pad 2: Net-(F1-Pad2) -> Net-(C17-Pad1)
- Q1 pad 3: Net-(C17-Pad1) -> Net-(F1-Pad2)
- U2 pad 55: /Ethernet/RXD0 -> Net-(TP2-Pad1)
- U2 pad 58: /Ethernet/RXD1 -> /Ethernet/RXD0
- U2 pad 59: /Ethernet/RXD2 -> /Ethernet/RXD1
- U2 pad 60: /Ethernet/RXD3 -> /Ethernet/RXD2
- U2 pad 64: Net-(U2-Pad64) -> /Ethernet/RXD3
- U2 pad 66: /Ethernet/TXD3 -> Net-(U2-Pad66)
- U2 pad 67: /Ethernet/TXD2 -> /Ethernet/TXD3
- U2 pad 68: /Ethernet/TXD1 -> /Ethernet/TXD2
- U2 pad 69: /Ethernet/TXD0 -> /Ethernet/TXD1
- U2 pad 71: Net-(DB7-Pad1) -> /Ethernet/TXD0
- U4 pad 24: Net-(U2-Pad65) -> Net-(U2-Pad66)
- U4 pad 25: Net-(U2-Pad64) -> Net-(U2-Pad65)
Routing:
- net GND: track 664.4 -> 997.5 mm, vias 210 -> 288
- net Net-(J29-Pad1): track 0.00 -> 56.9 mm, vias 0 -> 2
- net +3V3: track 572.4 -> 616.7 mm, vias 38 -> 40
- net Net-(U2-Pad64): track 11.0 -> 0.00 mm
- net Net-(B121-Pad1): track 0.00 -> 10.3 mm
- net +VPA: track 161.0 -> 171.3 mm, vias 6 -> 9
- net Net-(U2-Pad66): track 0.00 -> 9.78 mm
- net Net-(DB7-Pad1): track 6.38 -> 0.00 mm
- net /PA/TR: track 68.6 -> 64.4 mm, vias 0 -> 1
- net Net-(B118-Pad1): track 7.59 -> 10.9 mm
- net Net-(TP2-Pad1): track 0.00 -> 2.79 mm
- net Net-(CN3-Pad13): track 35.0 -> 33.0 mm
- net Net-(U2-Pad65): track 9.57 -> 11.3 mm
- net Net-(C81-Pad1): track 34.0 -> 32.8 mm
- net Net-(B97-Pad1): track 23.1 -> 24.1 mm
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Other:
- outline, holes or cut-outs redrawn

Commit message: Commit for printing
Parts:
- R43, R44: moved to F.Cu
- moved CL2 24.3 mm to (94.6, 125.0)
- moved R43 9.03 mm to (99.5, 112.2)
- moved R44 9.03 mm to (99.5, 115.0)
- moved B115 8.41 mm to (92.1, 108.6)
- moved B56 8.41 mm to (86.1, 112.1)
- moved B57 8.41 mm to (92.6, 110.8)
- moved B59 8.41 mm to (89.4, 102.3)
- moved B61 8.41 mm to (89.3, 107.8)
- moved B62 8.41 mm to (94.2, 106.0)
- moved B64 8.41 mm to (83.9, 104.3)
- moved C12 8.41 mm to (89.3, 104.3)
- moved C41 8.41 mm to (85.4, 110.3)
- moved C42 8.41 mm to (94.7, 112.5)
- moved C44 8.41 mm to (94.2, 107.6)
- moved FB12 8.41 mm to (85.4, 108.6)
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Routing:
- net Net-(CL2-Pad1): track 11.2 -> 31.8 mm, vias 0 -> 1
- net /Clock/SCL1: track 49.6 -> 40.7 mm
- net /Clock/SDA1: track 47.2 -> 39.2 mm
- net Net-(B58-Pad2): track 3.84 -> 10.2 mm
- net Net-(B58-Pad1): track 12.4 -> 6.92 mm
- net Net-(J23-Pad1): track 44.3 -> 39.6 mm
- net +3V3: track 616.7 -> 618.1 mm
- net RFFE_CLK: track 28.0 -> 29.3 mm
- net Net-(B65-Pad2): track 31.6 -> 32.3 mm

Commit message: Before ethernet phy rework
Routing:
- net GND: track 997.5 -> 995.0 mm
Changed lines of the file:
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@@
     (area 31.849999 38.7 205.090477 152.071428)
     (thickness 1.6)
-    (drawings 77)
-    (tracks 4899)
+    (drawings 69)
+    (tracks 4898)
     (zones 0)
     (modules 516)
@@
   (title_block
     (title "Hermes-Lite 2.0")
-    (date 2016-10-30)
+    (date 2016-11-06)
     (rev 2.0-beta1)
     (company SofterHardware)
@@
   (gr_line (start 120.2 126.9) (end 120.2 125.6) (angle 90) (layer B.SilkS) (width 0.1))
   (gr_line (start 120.5 127.2) (end 120.2 126.9) (angle 90) (layer B.SilkS) (width 0.1))
-  (gr_line (start 38.1 122.8) (end 38.5 122.4) (angle 90) (layer B.SilkS) (width 0.1))
-  (gr_line (start 38.1 115.8) (end 38.1 114.9) (angle 90) (layer B.SilkS) (width 0.1))
-  (gr_line (start 37.3 115.8) (end 38.1 115.8) (angle 90) (layer B.SilkS) (width 0.1))
-  (gr_line (start 37.7 111.8) (end 38.2 111.3) (angle 90) (layer B.SilkS) (width 0.1))
-  (gr_line (start 37.7 113.4) (end 37.7 111.8) (angle 90) (layer B.SilkS) (width 0.1))
-  (gr_line (start 37.4 113.7) (end 37.7 113.4) (angle 90) (layer B.SilkS) (width 0.1))
-  (gr_line (start 39.2 119.7) (end 39.2 120.5) (angle 90) (layer B.SilkS) (width 0.1))
-  (gr_line (start 32.3 114.9) (end 31.9 115.3) (angle 90) (layer B.SilkS) (width 0.1))
   (gr_line (start 110.6 112.5) (end 111 112.9) (angle 90) (layer B.SilkS) (width 0.1))
   (gr_line (start 119.1 114.7) (end 120.9 114.7) (angle 90) (layer B.SilkS) (width 0.1))
@@
   (segment (start 97.5 139) (end 100 139) (width 0.35) (layer F.Cu) (net 31))
   (via (at 100 139) (size 0.8) (drill 0.5) (layers F.Cu B.Cu) (net 31))
-  (segment (start 100 139) (end 102.5 139) (width 0.35) (layer B.Cu) (net 31))
   (via (at 102.5 139) (size 0.8) (drill 0.5) (layers F.Cu B.Cu) (net 31))
   (segment (start 102.5 139) (end 105 139) (width 0.35) (layer F.Cu) (net 31))

Commit message: Hermes-Lite 2.0beta2
Parts:
- moved R31 13.3 mm to (107.3, 51.6)
- moved R20 6.58 mm to (110.0, 54.7), turned to 180 degrees
- moved B51 4.79 mm to (95.6, 66.8)
- moved C39 3.80 mm to (110.4, 51.1)
- moved FB10 3.80 mm to (113.2, 50.7)
- moved FB29 3.80 mm to (113.2, 52.3)
- moved R27 3.41 mm to (110.0, 56.3)
- moved R25 2.67 mm to (108.4, 61.8), turned to 180 degrees
- moved B52 2.22 mm to (102.7, 59.6)
- moved B45 2.18 mm to (97.7, 65.0), turned to 90 degrees
- moved R26 1.91 mm to (110.0, 57.9), turned to 180 degrees
- moved R28 1.41 mm to (108.4, 60.2), turned to 0 degrees
- moved B53 0.72 mm to (100.5, 57.9), turned to 270 degrees
- moved C38 0.70 mm to (100.7, 51.9)
- moved B42 0.64 mm to (95.6, 57.9), turned to 270 degrees
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Routing:
- net GND: track 995.0 -> 1240.1 mm, vias 288 -> 278
- net Net-(CN3-Pad16): track 20.0 -> 34.2 mm
- net Net-(B42-Pad1): track 30.9 -> 39.8 mm
- net +1V2: track 186.3 -> 192.2 mm, vias 27 -> 29
- net Veth: track 102.1 -> 98.0 mm
- net +3V3: track 618.1 -> 614.3 mm
- net Net-(R27-Pad1): track 27.2 -> 30.7 mm
- net Net-(C35-Pad1): track 23.1 -> 25.2 mm
- net Net-(CN3-Pad17): track 44.7 -> 46.7 mm
- net Net-(B40-Pad1): track 22.8 -> 24.6 mm, vias 4 -> 3
- net Net-(CN3-Pad13): track 33.0 -> 34.6 mm
- net Net-(R20-Pad2): track 11.5 -> 9.90 mm
- net /Ethernet/RXD3: track 13.4 -> 14.6 mm
- net Net-(R26-Pad2): track 25.7 -> 24.7 mm
- net Net-(R34-Pad1): track 6.33 -> 7.25 mm
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Other:
- outline, holes or cut-outs redrawn
- board text added: "Hermes-Lite 2.0-beta2 © 2016 SofterHardware"
- board text removed: "Hermes-Lite 2.0-beta1 © 2016 SofterHardware"
